File: pcb/single-board/bytecradle-6502-single-board.kicad_sch (KiCad schematic)
At the start: 53 parts, among them J1 BUS, J2 USB_B, J3 Serial, SW1 SW_DIP_x04, SW2 RESET, SW3 NMI, U1 W65C02SxP, U10 74HC688, U11 74HC32, U12 74HC688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

Commit message: Initial lay-out PCB
Parts:
- added C20, C21: 100nF, Capacitor_THT:C_Disc_D5.0mm_W2.5mm_P5.00mm, symbol Device:C
- added U18: 74HC00, Package_DIP:DIP-14_W7.62mm_Socket, symbol 74xx:74HC00
- C1: value C -> 30pF; footprint (none) -> Capacitor_THT:C_Disc_D5.0mm_W2.5mm_P5.00mm
- C10, C11, C12, C13, C14, C15, C16, C17, C2, C3, C4, C5, C6, C7, C8, C9: footprint (none) -> Capacitor_THT:C_Disc_D5.0mm_W2.5mm_P5.00mm
- C18, C19: footprint Capacitor_SMD:CP_Elec_6.3x3.9 -> Capacitor_THT:CP_Radial_D6.3mm_P2.50mm
- D1: footprint (none) -> LED_THT:LED_D5.0mm
- J3: footprint (none) -> Connector_PinSocket_2.54mm:PinSocket_1x06_P2.54mm_Vertical
- R1, R2, R3: footprint (none) -> Resistor_THT:R_Axial_DIN0207_L6.3mm_D2.5mm_P7.62mm_Horizontal
- SW1: footprint (none) -> Button_Switch_THT:SW_DIP_SPSTx04_Slide_9.78x12.34mm_W7.62mm_P2.54mm
- U10, U12, U17, U3, U4, U9: footprint (none) -> Package_DIP:DIP-20_W7.62mm_Socket
- U11, U16, U6: footprint (none) -> Package_DIP:DIP-14_W7.62mm_Socket
- U14, U15: footprint (none) -> Package_DIP:DIP-16_W7.62mm_Socket
- U2: footprint (none) -> Package_DIP:DIP-32_W15.24mm_Socket
- Y1: footprint (none) -> Crystal:Crystal_HC50_Horizontal
Connections:
- net A15: no longer U7.22 (~{OE})
- net CLK: now also U6.13, U18.2
- net GND: now also C20.2, C21.2, U18.10, U18.12, U18.13, U18.7 (GND), U18.9
- net R/~{W}: no longer U7.27 (~{WE}), U8.27 (~{WE})
- net VCC: now also C20.1, C21.1, U18.14 (VCC)
- net ~{R}/W: now also U11.1, U6.12, U7.22 (~{OE}), U8.22 (~{OE}); no longer U11.2
- net at U3.11 (Cp): now also U18.3; no longer U6.11
- net at U11.8, U8.20 (~{CS}): no longer U8.22 (~{OE})
- net at U10.19 (P=R), U11.5: now also U11.2; no longer U11.1
- new net: U11.6, U18.4, U18.5
- new net: U18.1, U18.6
- new net: U6.11, U7.27 (~{WE}), U8.27 (~{WE})
- no-connect marks 34 -> 36
Other:
- moved on the sheet: U11C, U11D, U6D

Commit message: Tuning design
Parts:
- J1: footprint (none) -> edgeconn:DIP-60_200_ELL
- RN1: value R_Network08 -> 10k
- U2: footprint Package_DIP:DIP-32_W15.24mm_Socket -> Socket:DIP_Socket-32_W11.9_W12.7_W15.24_W17.78_W18.5_3M_232-1285-00-0602J
- Y1: value Crystal -> 1.8432 MHz; footprint Crystal:Crystal_HC50_Horizontal -> Crystal:Crystal_HC50_Vertical
Changed lines of the file:
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@@
 			)
 		)
-		(property "Footprint" "Package_DIP:DIP-32_W15.24mm_Socket"
+		(property "Footprint" "Socket:DIP_Socket-32_W11.9_W12.7_W15.24_W17.78_W18.5_3M_232-1285-00-0602J"
 			(at 346.71 63.5 0)
 			(effects
@@
 			)
 		)
-		(property "Value" "Crystal"
+		(property "Value" "1.8432 MHz"
 			(at 113.03 213.3599 90)
 			(effects
@@
 			)
 		)
-		(property "Footprint" "Crystal:Crystal_HC50_Horizontal"
+		(property "Footprint" "Crystal:Crystal_HC50_Vertical"
 			(at 109.22 212.09 0)
 			(effects
@@
 			)
 		)
-		(property "Footprint" ""
+		(property "Footprint" "edgeconn:DIP-60_200_ELL"
 			(at 243.84 237.49 0)
 			(effects
@@
 			)
 		)
-		(property "Value" "R_Network08"
+		(property "Value" "10k"
 			(at 35.814 129.54 90)
 			(effects
