File: pcb/single-board/bytecradle-6502-single-board.kicad_sch (KiCad schematic)
At the start: 62 parts, among them J1 BUS, J2 USB_B, J3 Serial, SW1 SW_DIP_x04, SW2 RESET, SW3 NMI, U1 W65C02SxP, U10 74HC688, U11 74HC02, U12 74HC688, U13 W65C22NxP, U14 74HC193, U15 74HC193, U16 74HC14, U17 74HC688, U18 74HC00, U19 74HC08, U2 SST39SF040, U3 74HC273, U4 74HC688, U5 W65C51NxP, U6 74HC00, U7 CY62256-70PC, U8 CY62256-70PC, U9 74HC245, X1 32MHz, Y1 1.8432 MHz

Commit message: Finalizing lay-out
Parts:
- added TP4: ~{NMI}, Connector_PinHeader_2.54mm:PinHeader_1x01_P2.54mm_Vertical, symbol Connector:TestPoint_Probe
- added TP5: ~{RES}, Connector_PinHeader_2.54mm:PinHeader_1x01_P2.54mm_Vertical, symbol Connector:TestPoint_Probe
- added TP6: ~{IRQ}, Connector_PinHeader_2.54mm:PinHeader_1x01_P2.54mm_Vertical, symbol Connector:TestPoint_Probe
- R6: value 220 -> 560
- SW1: value SW_DIP_x04 -> CLOCKDIV
Connections:
- net GND: no longer J1.30 (Pin_30)
- net ~{IRQ}: now also TP6.1
- net ~{NMI}: now also J1.30 (Pin_30), TP4.1
- net ~{RES}: now also TP5.1
Other:
- note added: "0x0000-0x7FFF (32 KiB)"
- note added: "0x8000-0xBFFF excl. 0x9FXX (~ 16 KiB)"
- note added: "0xC000-0xFFFF (16 KiB)"
- note added: "Latch LOW-to-HIGH Happens when CLK goes low"
- note removed: "0x0000-0x7FFF"
- note removed: "0x8000-0xBFFF excl. 0x9FXX"
- note removed: "0xC000-0xFFFF"
- note removed: "Latch on descending edge"
- moved on the sheet: TP1, TP2, TP3

Commit message: Adding Arduino interface and test code for ACIA
Parts:
- added R2, R8: 1k, Resistor_THT:R_Axial_DIN0207_L6.3mm_D2.5mm_P7.62mm_Horizontal, symbol Device:R
Connections:
- net GND: no longer U5.16 (~{DCD}), U5.17 (~{DSR})
- net VCC: now also R2.2, R8.1
- net ~{IRQC22}: now also R8.2
- net ~{IRQC51}: now also R2.1
- no-connect marks 36 -> 38

Commit message: Refining PCBs
Parts:
- removed C24: 100nF, Capacitor_THT:C_Disc_D5.0mm_W2.5mm_P5.00mm, symbol Device:C
- removed J1: BUS, edgeconn:DIP-60_200_ELL, symbol Connector_Generic:Conn_02x30_Counter_Clockwise
- removed RN1: 10k, Resistor_THT:R_Array_SIP9, symbol Device:R_Network08
- removed SW1: CLOCKDIV, Button_Switch_THT:SW_DIP_SPSTx04_Slide_9.78x12.34mm_W7.62mm_P2.54mm, symbol Switch:SW_DIP_x04
- removed U14, U15: 74HC193, Package_DIP:DIP-16_W7.62mm_Socket, symbol 74xx:74LS193
- removed U8: CY62256-70PC, Package_DIP:DIP-28_W15.24mm_Socket, symbol Memory_RAM:CY62256-70PC
- added C25, C26, C27, C28, C30, C31: 100nF, Capacitor_THT:C_Disc_D5.0mm_W2.5mm_P5.00mm, symbol Device:C
- added C29: 30pF, Capacitor_THT:C_Disc_D5.0mm_W2.5mm_P5.00mm, symbol Device:C
- added H1, H2, H3, H4: MountingHole, MountingHole:MountingHole_3.2mm_M3, symbol Mechanical:MountingHole
- added J1: VIA, Connector_PinHeader_2.54mm:PinHeader_2x20_P2.54mm_Vertical, symbol Connector_Generic:Conn_02x20_Counter_Clockwise
- added J4: Serial, Connector_PinSocket_2.54mm:PinSocket_1x06_P2.54mm_Vertical, symbol Connector:Conn_01x06_Socket
- added J5: EXPBUS1, Connector_PinHeader_2.54mm:PinHeader_2x20_P2.54mm_Vertical, symbol Connector_Generic:Conn_02x20_Counter_Clockwise
- added J6: EXPBUS2, Connector_PinHeader_2.54mm:PinHeader_2x20_P2.54mm_Vertical, symbol Connector_Generic:Conn_02x20_Counter_Clockwise
- added J7: UART1, Connector_Dsub:DSUB-9_Male_Horizontal_P2.77x2.84mm_EdgePinOffset4.94mm_Housed_MountingHolesOffset7.48mm, symbol Connector:DE9_Plug_MountingHoles
- added J8: UART2, Connector_Dsub:DSUB-9_Male_Horizontal_P2.77x2.84mm_EdgePinOffset4.94mm_Housed_MountingHolesOffset7.48mm, symbol Connector:DE9_Plug_MountingHoles
- added R10: 1M, Resistor_THT:R_Axial_DIN0207_L6.3mm_D2.5mm_P7.62mm_Horizontal, symbol Device:R
- added R9: 1k, Resistor_THT:R_Axial_DIN0207_L6.3mm_D2.5mm_P7.62mm_Horizontal, symbol Device:R
- added U14: 74HC273, Package_DIP:DIP-20_W7.62mm_Socket, symbol 74xx:74AHC273
- added U15: 74HC245, Package_DIP:DIP-20_W7.62mm_Socket, symbol 74xx:74HC245
- added U20, U22: 74HC688, Package_DIP:DIP-20_W7.62mm_Socket, symbol 74xx:74HC688
- added U21: 74HC02, Package_DIP:DIP-14_W7.62mm_Socket, symbol 74xx:74HC02
- added U23: W65C51NxP, Package_DIP:DIP-28_W15.24mm_Socket, symbol 65xx-library:W65C51NxP
- added U8: AS6C4008-55PCN, Package_DIP:DIP-32_W15.24mm, symbol Memory_RAM:AS6C4008-55PCN
- added Y2: 1.8432 MHz, Crystal:Crystal_HC50_Vertical, symbol Device:Crystal
Connections:
- net A0: now also J5.2 (Pin_2), J6.2 (Pin_2), U20.2 (P0), U23.13 (RS0), U8.12 (A0)
- net A1: now also J5.3 (Pin_3), J6.3 (Pin_3), U20.4 (P1), U23.14 (RS1), U8.11 (A1)
- net A10: now also J5.12 (Pin_12), J6.12 (Pin_12), U8.23 (A10)
- net A11: now also J5.13 (Pin_13), J6.13 (Pin_13), U8.25 (A11)
- net A12: now also J5.14 (Pin_14), J6.14 (Pin_14), U8.4 (A12)
- net A13: now also J5.15 (Pin_15), J6.15 (Pin_15), U8.28 (A13)
- net A14: now also J5.16 (Pin_16), J6.16 (Pin_16)
- net A15: now also J5.17 (Pin_17), J6.17 (Pin_17)
- net A2: now also J5.4 (Pin_4), J6.4 (Pin_4), U20.6 (P2), U22.6 (P2), U8.10 (A2)
- net A3: now also J5.5 (Pin_5), J6.5 (Pin_5), U20.8 (P3), U22.8 (P3), U8.9 (A3)
- net A4: now also J5.6 (Pin_6), J6.6 (Pin_6), U20.11 (P4), U22.11 (P4), U8.8 (A4)
- net A5: now also J5.7 (Pin_7), J6.7 (Pin_7), U20.13 (P5), U22.13 (P5), U8.7 (A5)
- net A6: now also J5.8 (Pin_8), J6.8 (Pin_8), U20.15 (P6), U22.15 (P6), U8.6 (A6)
- net A7: now also J5.9 (Pin_9), J6.9 (Pin_9), U20.17 (P7), U22.17 (P7), U8.5 (A7)
- net A8: now also J5.10 (Pin_10), J6.10 (Pin_10), U8.27 (A8)
- net A9: now also J5.11 (Pin_11), J6.11 (Pin_11), U8.26 (A9)
- net CA1: now also J1.39 (Pin_39)
- net CA2: now also J1.38 (Pin_38)
- net CB1: now also J1.37 (Pin_37)
- net CB2: now also J1.36 (Pin_36)
- net CLK: now also U6.5, J1.22 (Pin_22), J5.38 (Pin_38), J6.38 (Pin_38), U23.27 (ϕ2)
- net D0: now also J5.29 (Pin_29), J6.29 (Pin_29), U14.3 (D0), U15.18 (B0), U23.18 (D0), U8.13 (DQ0)
- net D1: now also J5.28 (Pin_28), J6.28 (Pin_28), U14.4 (D1), U15.17 (B1), U23.19 (D1), U8.14 (DQ1)
- net D2: now also J5.27 (Pin_27), J6.27 (Pin_27), U14.7 (D2), U15.16 (B2), U23.20 (D2), U8.15 (DQ2)
- net D3: now also J5.26 (Pin_26), J6.26 (Pin_26), U14.8 (D3), U15.15 (B3), U23.21 (D3), U8.17 (DQ3)
- net D4: now also J5.25 (Pin_25), J6.25 (Pin_25), U14.13 (D4), U15.14 (B4), U23.22 (D4), U8.18 (DQ4)
- net D5: now also J5.24 (Pin_24), J6.24 (Pin_24), U14.14 (D5), U15.13 (B5), U23.23 (D5), U8.19 (DQ5)
- net D6: now also J5.23 (Pin_23), J6.23 (Pin_23), U14.17 (D6), U15.12 (B6), U23.24 (D6), U8.20 (DQ6)
- net D7: now also J5.22 (Pin_22), J6.22 (Pin_22), U14.18 (D7), U15.11 (B7), U23.25 (D7), U8.21 (DQ7)
- net GND: now also C25.2, C26.2, C27.2, C28.2, C29.1, C30.2, C31.2, J1.10 (Pin_10), J1.11 (Pin_11), J1.20 (Pin_20), J1.21 (Pin_21), J4.6 (Pin_6), J5.20 (Pin_20), J5.21 (Pin_21), J6.20 (Pin_20), J6.21 (Pin_21), J7.5, J8.5, U14.10 (GND), U15.10 (GND), U20.10 (GND), U20.12 (R4), U20.14 (R5), U20.16 (R6), U20.18 (R7), U20.5 (R1), U20.7 (R2), U20.9 (R3), U21.7 (GND), U22.10 (GND), U22.12 (R4), U22.14 (R5), U22.16 (R6), U22.18 (R7), U22.2 (P0), U22.3 (R0), U22.4 (P1), U22.5 (R1), U22.7 (R2), U23.1 (VSS), U8.16 (VSS); no longer U19.10, U19.12, U19.13, U19.9, U6.4, U6.5
- net PA0: now also J1.2 (Pin_2)
- net PA1: now also J1.3 (Pin_3)
- net PA2: now also J1.4 (Pin_4)
- net PA3: now also J1.5 (Pin_5)
- net PA4: now also J1.6 (Pin_6)
- net PA5: now also J1.7 (Pin_7)
- net PA6: now also J1.8 (Pin_8)
- net PA7: now also J1.9 (Pin_9)
- net PB0: now also J1.12 (Pin_12)
- net PB1: now also J1.13 (Pin_13)
- net PB2: now also J1.14 (Pin_14)
- net PB3: now also J1.15 (Pin_15)
- net PB4: now also J1.16 (Pin_16)
- net PB5: now also J1.17 (Pin_17)
- net PB6: now also J1.18 (Pin_18)
- net PB7: now also J1.19 (Pin_19)
- net R/~{W}: now also J1.23 (Pin_23), J5.39 (Pin_39), J6.39 (Pin_39), U21.2, U21.3, U21.5, U23.28 (R/~{W}), U8.29 (WE#)
- net VCC: now also U19.13, C25.1, C26.1, C27.1, C28.1, C30.1, C31.1, J1.1 (Pin_1), J1.40 (Pin_40), J4.4 (Pin_4), J5.1 (Pin_1), J5.40 (Pin_40), J6.1 (Pin_1), J6.40 (Pin_40), R9.2, U14.20 (VCC), U15.1 (A->B), U15.20 (VCC), U20.20 (VCC), U20.3 (R0), U21.14 (VCC), U22.20 (VCC), U22.9 (R3), U23.15 (VCC), U23.2 (CS1), U8.32 (VCC)
- net ~{IRQC22}: now also J1.33 (Pin_33)
- net ~{IRQ}: now also U19.8, J5.34 (Pin_34), J6.34 (Pin_34); no longer U19.3
- net ~{I/O}: now also J1.34 (Pin_34), J5.32 (Pin_32), J6.32 (Pin_32), U20.1 (G), U22.1 (G)
- net ~{NMI}: now also J1.32 (Pin_32), J5.35 (Pin_35), J6.35 (Pin_35)
- net ~{RES}: now also J1.35 (Pin_35), J5.36 (Pin_36), J6.36 (Pin_36), U14.1 (~{Mr}), U23.4 (~{RES})
- net at X1.8 (OUT): now also U16.1
- net at U11.1: now also U8.24 (OE#)
- net at U19.11: now also U19.10
- net at U18.8: now also U8.22 (CE#)
- net at U6.6: now also U14.11 (Cp)
- net BANK0: no longer names the net of U2.29 (A14), U3.2 (Q0), U9.2 (A0)
- net BANK1: no longer names the net of U2.3 (A15), U3.5 (Q1), U9.3 (A1)
- net BANK2: no longer names the net of U2.2 (A16), U3.6 (Q2), U9.4 (A2)
- net BANK3: no longer names the net of U2.30 (A17), U3.9 (Q3), U9.5 (A3)
- net BANK4: no longer names the net of U2.1 (A18), U3.12 (Q4), U9.6 (A4)
- net RAMBANK: no longer names the net of U3.15 (Q5), U9.7 (A5)
- net REG6: no longer names the net of U3.16 (Q6), U9.8 (A6)
- net REG7: no longer names the net of U3.19 (Q7), U9.9 (A7)
- net RxD renamed RxD1
- net RxD1: now also J1.29 (Pin_29), J7.3
- net TxD renamed TxD1
- net TxD1: now also J1.30 (Pin_30), J7.2
- net ~{CTS} renamed ~{CTS1}
- net ~{CTS1}: now also J1.28 (Pin_28), J7.7
- net ~{IRQC51} renamed ~{IRQC51_1}
- net ~{RTS} renamed ~{RTS1}
- net ~{RTS1}: now also J1.31 (Pin_31), J7.8
- new net: U19.3, U19.9
- new net: U21.10, U21.11, U21.12
- new net: U15.19 (CE), U21.13
- new net: U21.1, U21.8
- new net: R10.2, U23.7 (XTAL2), Y2.1
- new net: C29.2, R10.1, U23.6 (XTAL1), Y2.2
- new net: U22.19 (P=R), U23.3 (~{CS2})
- new net: U14.12 (Q4), U15.6 (A4), U8.1 (A18)
- new net: U14.6 (Q2), U15.4 (A2), U8.2 (A16)
- new net: U14.2 (Q0), U15.2 (A0), U8.3 (A14)
- new net: U14.9 (Q3), U15.5 (A3), U8.30 (A17)
- new net: U14.5 (Q1), U15.3 (A1), U8.31 (A15)
- new net: U21.4, U6.4
- new net: U20.19 (P=R), U21.6, U21.9
- new net: U14.15 (Q5), U15.7 (A5)
- new net: U14.16 (Q6), U15.8 (A6)
- new net: U14.19 (Q7), U15.9 (A7)
- new net RxD2: J1.25 (Pin_25), J4.3 (Pin_3), J8.3, U23.12 (RxD)
- new net TxD2: J1.26 (Pin_26), J4.2 (Pin_2), J8.2, U23.10 (TxD)
- new net ~{CTS2}: J1.24 (Pin_24), J4.5 (Pin_5), J8.7, U23.9 (~{CTS})
- new net ~{IRQC51_2}: R9.1, U19.12, U23.26 (~{IRQ})
- new net ~{RTS2}: J1.27 (Pin_27), J4.1 (Pin_1), J8.8, U23.8 (~{RTS})
- no-connect marks 38 -> 43
Other:
- note added: "0x9F01"
- note added: "0x9F08-0x9F0B"
- note added: "CPU and CLOCK"
- note added: "HIGH MEMORY"
- note added: "LOW MEMORY"
- note added: "ROM"
- note added: "ROM / RAM including BANKING"
- note added: "UART 1"
- note added: "UART 2"
- moved on the sheet: C10, C11, C12, C13, C20, C21, C7, C8, C9, R1, R8, U1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

Commit message: Further redesigning boards
Parts:
- removed C1, C29: 30pF, Capacitor_THT:C_Disc_D5.0mm_W2.5mm_P5.00mm, symbol Device:C
- removed C10, C11, C12, C13, C14, C15, C16, C17, C20, C21, C25, C26, C27, C28, C30, C31, C7, C8, C9: 100nF, Capacitor_THT:C_Disc_D5.0mm_W2.5mm_P5.00mm, symbol Device:C
- removed J1: VIA, Connector_PinHeader_2.54mm:PinHeader_2x20_P2.54mm_Vertical, symbol Connector_Generic:Conn_02x20_Counter_Clockwise
- removed J3, J4: Serial, Connector_PinSocket_2.54mm:PinSocket_1x06_P2.54mm_Vertical, symbol Connector:Conn_01x06_Socket
- removed J7: UART1, Connector_Dsub:DSUB-9_Male_Horizontal_P2.77x2.84mm_EdgePinOffset4.94mm_Housed_MountingHolesOffset7.48mm, symbol Connector:DE9_Plug_MountingHoles
- removed J8: UART2, Connector_Dsub:DSUB-9_Male_Horizontal_P2.77x2.84mm_EdgePinOffset4.94mm_Housed_MountingHolesOffset7.48mm, symbol Connector:DE9_Plug_MountingHoles
- removed R10, R3: 1M, Resistor_THT:R_Axial_DIN0207_L6.3mm_D2.5mm_P7.62mm_Horizontal, symbol Device:R
- removed R2, R8, R9: 1k, Resistor_THT:R_Axial_DIN0207_L6.3mm_D2.5mm_P7.62mm_Horizontal, symbol Device:R
- removed U10, U12, U17, U20, U22: 74HC688, Package_DIP:DIP-20_W7.62mm_Socket, symbol 74xx:74HC688
- removed U11, U21: 74HC02, Package_DIP:DIP-14_W7.62mm_Socket, symbol 74xx:74HC02
- removed U13: W65C22NxP, Package_DIP:DIP-40_W15.24mm_Socket, symbol 65xx-library:W65C22NxP
- removed U14, U3: 74HC273, Package_DIP:DIP-20_W7.62mm_Socket, symbol 74xx:74AHC273
- removed U15, U9: 74HC245, Package_DIP:DIP-20_W7.62mm_Socket, symbol 74xx:74HC245
- removed U18, U6: 74HC00, Package_DIP:DIP-14_W7.62mm_Socket, symbol 74xx:74HC00
- removed U2: SST39SF040, Socket:DIP_Socket-32_W11.9_W12.7_W15.24_W17.78_W18.5_3M_232-1285-00-0602J, symbol Memory_Flash:SST39SF040
- removed U23, U5: W65C51NxP, Package_DIP:DIP-28_W15.24mm_Socket, symbol 65xx-library:W65C51NxP
- removed U7: CY62256-70PC, Package_DIP:DIP-28_W15.24mm_Socket, symbol Memory_RAM:CY62256-70PC
- removed U8: AS6C4008-55PCN, Package_DIP:DIP-32_W15.24mm, symbol Memory_RAM:AS6C4008-55PCN
- removed Y1, Y2: 1.8432 MHz, Crystal:Crystal_HC50_Vertical, symbol Device:Crystal
- added SW1: SW_SPDT, components:power_switch, symbol Switch:SW_SPDT
- J2: renamed from J5; symbol Connector_Generic:Conn_02x20_Counter_Clockwise -> Connector_Generic:Conn_02x20_Odd_Even
- J3: renamed from J6; symbol Connector_Generic:Conn_02x20_Counter_Clockwise -> Connector_Generic:Conn_02x20_Odd_Even
- U2: renamed from U1; value W65C02SxP -> W65C02
- renumbered C2 to C1, C3 to C2, C6 to C3, C5 to C4, C4 to C5, C18 to C6, C19 to C7, C22 to C8, C23 to C9, J2 to J1, R4 to R2, R6 to R3, R5 to R4, R7 to R5, U16 to U1, U4 to U3, U19 to U4
Connections:
- net A0: now also J2.3 (Pin_3), J3.3 (Pin_3); no longer J2.2 (Pin_2), J3.2 (Pin_2)
- net A1: now also J2.5 (Pin_5), J3.5 (Pin_5); no longer J2.3 (Pin_3), J3.3 (Pin_3)
- net A10: now also J2.23 (Pin_23), J3.23 (Pin_23); no longer J2.12 (Pin_12), J3.12 (Pin_12)
- net A11: now also J2.25 (Pin_25), J3.25 (Pin_25); no longer J2.13 (Pin_13), J3.13 (Pin_13)
- net A12: now also J2.27 (Pin_27), J3.27 (Pin_27); no longer J2.14 (Pin_14), J3.14 (Pin_14)
- net A13: now also J2.29 (Pin_29), J3.29 (Pin_29); no longer J2.15 (Pin_15), J3.15 (Pin_15)
- net A14: now also J2.31 (Pin_31), J3.31 (Pin_31); no longer J2.16 (Pin_16), J3.16 (Pin_16)
- net A15: now also J2.33 (Pin_33), J3.33 (Pin_33); no longer J2.17 (Pin_17), J3.17 (Pin_17)
- net A2: now also J2.7 (Pin_7), J3.7 (Pin_7); no longer J2.4 (Pin_4), J3.4 (Pin_4)
- net A3: now also J2.9 (Pin_9), J3.9 (Pin_9); no longer J2.5 (Pin_5), J3.5 (Pin_5)
- net A4: now also J2.11 (Pin_11), J3.11 (Pin_11); no longer J2.6 (Pin_6), J3.6 (Pin_6)
- net A5: now also J2.13 (Pin_13), J3.13 (Pin_13); no longer J2.7 (Pin_7), J3.7 (Pin_7)
- net A6: now also J2.15 (Pin_15), J3.15 (Pin_15); no longer J2.8 (Pin_8), J3.8 (Pin_8)
- net A7: now also J2.17 (Pin_17), J3.17 (Pin_17); no longer J2.9 (Pin_9), J3.9 (Pin_9)
- net A8: now also J2.19 (Pin_19), J3.19 (Pin_19); no longer J2.10 (Pin_10), J3.10 (Pin_10)
- net A9: now also J2.21 (Pin_21), J3.21 (Pin_21); no longer J2.11 (Pin_11), J3.11 (Pin_11)
- net CLK: now also J2.6 (Pin_6), J3.6 (Pin_6); no longer J2.38 (Pin_38), J3.38 (Pin_38)
- net D0: now also J2.24 (Pin_24), J3.24 (Pin_24); no longer J2.29 (Pin_29), J3.29 (Pin_29)
- net D1: now also J2.26 (Pin_26), J3.26 (Pin_26); no longer J2.28 (Pin_28), J3.28 (Pin_28)
- net D2: now also J2.28 (Pin_28), J3.28 (Pin_28); no longer J2.27 (Pin_27), J3.27 (Pin_27)
- net D3: now also J2.30 (Pin_30), J3.30 (Pin_30); no longer J2.26 (Pin_26), J3.26 (Pin_26)
- net D4: now also J2.32 (Pin_32), J3.32 (Pin_32); no longer J2.25 (Pin_25), J3.25 (Pin_25)
- net D5: now also J2.34 (Pin_34), J3.34 (Pin_34); no longer J2.24 (Pin_24), J3.24 (Pin_24)
- net D6: now also J2.36 (Pin_36), J3.36 (Pin_36); no longer J2.23 (Pin_23), J3.23 (Pin_23)
- net D7: now also J2.38 (Pin_38), J3.38 (Pin_38); no longer J2.22 (Pin_22), J3.22 (Pin_22)
- net GND: now also J2.39 (Pin_39), J2.40 (Pin_40), J3.39 (Pin_39), J3.40 (Pin_40), U3.18 (R7); no longer J2.20 (Pin_20), J2.21 (Pin_21), J3.20 (Pin_20), J3.21 (Pin_21), U3.14 (R5), U3.16 (R6)
- net R/~{W}: now also J2.4 (Pin_4), J3.4 (Pin_4); no longer J2.39 (Pin_39), J3.39 (Pin_39)
- net VCC: now also J2.2 (Pin_2), J3.2 (Pin_2), U3.14 (R5), U3.16 (R6), SW1.1 (A); no longer J1.1 (VBUS), J2.40 (Pin_40), J3.40 (Pin_40), U3.18 (R7)
- net ~{IRQ}: now also J2.14 (Pin_14), J3.14 (Pin_14); no longer J2.34 (Pin_34), J3.34 (Pin_34)
- net ~{I/O}: now also J2.18 (Pin_18), J3.18 (Pin_18); no longer J2.32 (Pin_32), J3.32 (Pin_32)
- net ~{NMI}: now also J2.12 (Pin_12), J3.12 (Pin_12); no longer J2.35 (Pin_35), J3.35 (Pin_35)
- net ~{RES}: now also J2.10 (Pin_10), J3.10 (Pin_10); no longer J2.36 (Pin_36), J3.36 (Pin_36)
- new net VIN: J1.1 (VBUS), SW1.2 (B)
- no-connect marks 43 -> 26
Other:
- added sheet romram (romram.kicad_sch)
- added sheet uart (uart.kicad_sch)
- added sheet via (via.kicad_sch)
- note added: "0x7F"
- note added: "0x7FXX"
- note removed: "0x0000-0x7FFF (32 KiB)"
- note removed: "0x8000-0xBFFF excl. 0x9FXX (~ 16 KiB)"
- note removed: "0x9F00"
- note removed: "0x9F01"
- note removed: "0x9F04-0x9F07"
- note removed: "0x9F08-0x9F0B"
- note removed: "0x9F10-0x9F1F"
- note removed: "0x9FXX"
- note removed: "0xC000-0xFFFF (16 KiB)"
- note removed: "32 banks"
- note removed: "HIGH MEMORY"
- note removed: "LOW MEMORY"
- note removed: "Latch LOW-to-HIGH Happens when CLK goes low"
- note removed: "ROM"
- note removed: "ROM / RAM including BANKING"
- note removed: "UART 1"
- note removed: "UART 2"
- title: (none) -> ByteCradle 6502 - CPU & CLOCK
- moved on the sheet: C1, C2, C3, C4, C5, C6, C7, C8, C9, D1, H1, H2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

Commit message: Further revising
Parts:
- X1: value 32MHz -> 14 MHz
Other:
- note added: "Board-wide power-switch"
- note added: "Logical OR construction: If any of the ~{IRQ} request goes low (active), the CPU's ~{IRQ} will be triggered."
- note added: "Power indicator LED"
- note added: "Reset and NMI buttons with simplistic debouncing using a .1uF capacitor."
- note added: "Schmidt inverters are used to clean the clock signal. Might require using 74AC21."
- note added: "Single 74HC688 is used to map 0x7F00 - 0x7FF as the I/O space."
- note added: "Unused gates are tied to GND"
- moved on the sheet: C2, C6, C7, C8, C9, D1, J1, R2, R3, R4, R5, SW1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

Commit message: Refactoring source
Parts:
- U1: value 74HC14 -> 74AC14
- U3: value 74HC688 -> CD74HC688
- U4: value 74HC08 -> 74AC08
Changed lines of the file:
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@@
 			)
 		)
-		(property "Value" "74HC14"
+		(property "Value" "74AC14"
 			(at 44.45 149.86 90)
 			(effects
@@
 			)
 		)
-		(property "Value" "74HC08"
+		(property "Value" "74AC08"
 			(at 157.4717 35.56 0)
 			(effects
@@
 			)
 		)
-		(property "Value" "74HC14"
+		(property "Value" "74AC14"
 			(at 49.53 129.54 0)
 			(effects
@@
 			)
 		)
-		(property "Value" "74HC08"
+		(property "Value" "74AC08"
 			(at 140.9617 43.18 0)
 			(effects
@@
 			)
 		)
-		(property "Value" "74HC08"
+		(property "Value" "74AC08"
 			(at 139.7 73.66 90)
 			(effects
@@
 			)
 		)
-		(property "Value" "74HC688"
+		(property "Value" "CD74HC688"
 			(at 110.49 36.8614 0)
 			(effects
@@
 			)
 		)
-		(property "Value" "74HC14"
+		(property "Value" "74AC14"
 			(at 162.56 168.91 0)
 			(effects
@@
 			)
 		)
-		(property "Value" "74HC08"
+		(property "Value" "74AC08"
 			(at 140.9617 27.94 0)
 			(effects
@@
 			)
 		)
-		(property "Value" "74HC14"
+		(property "Value" "74AC14"
 			(at 134.62 184.15 0)
 			(effects
@@
 			)
 		)
-		(property "Value" "74HC14"
+		(property "Value" "74AC14"
 			(at 162.56 184.15 0)
 			(effects
@@
 			)
 		)
-		(property "Value" "74HC14"
+		(property "Value" "74AC14"
 			(at 64.77 129.54 0)
 			(effects
@@
 			)
 		)
-		(property "Value" "74HC08"
+		(property "Value" "74AC08"
 			(at 134.6117 168.91 0)
 			(effects
@@
 			)
 		)
-		(property "Value" "74HC14"
+		(property "Value" "74AC14"
 			(at 85.09 129.54 0)
 			(effects
