File: pcb/single-board/_autosave-bytecradle-6502-single-board.kicad_sch (KiCad schematic)
At the start: 62 parts, among them J1 BUS, J2 USB_B, J3 Serial, SW1 SW_DIP_x04, SW2 RESET, SW3 NMI, U1 W65C02SxP, U10 74HC688, U11 74HC02, U12 74HC688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

Commit message: Pre-routing commit
Parts:
- R6: value 220 -> 560
Changed lines of the file:
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@@
 			)
 		)
-		(property "Value" "220"
+		(property "Value" "560"
 			(at 319.786 232.41 90)
 			(effects
