File: pcb/single-board/bytecradle-6502-single-board.kicad_pcb (KiCad board)
At the start: 4 copper layers, 157.5 x 119.4 mm, 65 parts, among them J1 BUS, J2 USB_B, J3 Serial, SW1 CLOCKDIV, SW2 RESET, SW3 NMI, U1 W65C02SxP, U10 74HC688, U11 74HC02, U12 74HC688, U13 W65C22NxP, U14 74HC193, U15 74HC193, U16 74HC14, U17 74HC688, U18 74HC00, U19 74HC08, U2 SST39SF040, U3 74HC273, U4 74HC688, U5 W65C51NxP, U6 74HC00, U7 CY62256-70PC, U8 CY62256-70PC, U9 74HC245, X1 32MHz, Y1 1.8432 MHz

Commit message: Refining PCBs
Parts:
- removed C24: 100nF, Capacitor_THT:C_Disc_D5.0mm_W2.5mm_P5.00mm
- removed RN1: 10k, Resistor_THT:R_Array_SIP9
- removed SW1: CLOCKDIV, Button_Switch_THT:SW_DIP_SPSTx04_Slide_9.78x12.34mm_W7.62mm_P2.54mm
- added C25: 100nF, Capacitor_THT:C_Disc_D5.0mm_W2.5mm_P5.00mm, F.Cu at (88.9, 127.5)
- added C26: 100nF, Capacitor_THT:C_Disc_D5.0mm_W2.5mm_P5.00mm, F.Cu at (189.0, 58.7)
- added C27: 100nF, Capacitor_THT:C_Disc_D5.0mm_W2.5mm_P5.00mm, F.Cu at (171.4, 127.0)
- added C28: 100nF, Capacitor_THT:C_Disc_D5.0mm_W2.5mm_P5.00mm, F.Cu at (184.1, 127.0)
- added C29: 30pF, Capacitor_THT:C_Disc_D5.0mm_W2.5mm_P5.00mm, F.Cu at (178.8, 58.7)
- added C30: 100nF, Capacitor_THT:C_Disc_D5.0mm_W2.5mm_P5.00mm, F.Cu at (46.8, 52.3)
- added C31: 100nF, Capacitor_THT:C_Disc_D5.0mm_W2.5mm_P5.00mm, F.Cu at (31.8, 132.8)
- added H1: MountingHole, MountingHole:MountingHole_3.2mm_M3, F.Cu at (25.7, 44.7)
- added H2: MountingHole, MountingHole:MountingHole_3.2mm_M3, F.Cu at (209.0, 44.5)
- added H3: MountingHole, MountingHole:MountingHole_3.2mm_M3, F.Cu at (25.4, 156.2)
- added H4: MountingHole, MountingHole:MountingHole_3.2mm_M3, F.Cu at (209.0, 156.0)
- added J4: Serial, Connector_PinSocket_2.54mm:PinSocket_1x06_P2.54mm_Vertical, F.Cu at (179.3, 83.8)
- added J5: EXPBUS1, Connector_PinHeader_2.54mm:PinHeader_2x20_P2.54mm_Vertical, F.Cu at (207.3, 53.3)
- added J6: EXPBUS2, Connector_PinHeader_2.54mm:PinHeader_2x20_P2.54mm_Vertical, F.Cu at (195.6, 106.7)
- added J7: UART1, Connector_Dsub:DSUB-9_Male_Horizontal_P2.77x2.84mm_EdgePinOffset4.94mm_Housed_MountingHolesOffset7.48mm, F.Cu at (144.7, 49.2)
- added J8: UART2, Connector_Dsub:DSUB-9_Male_Horizontal_P2.77x2.84mm_EdgePinOffset4.94mm_Housed_MountingHolesOffset7.48mm, F.Cu at (192.2, 49.3)
- added R10: 1M, Resistor_THT:R_Axial_DIN0207_L6.3mm_D2.5mm_P7.62mm_Horizontal, F.Cu at (172.2, 70.1)
- added R2: 1k, Resistor_THT:R_Axial_DIN0207_L6.3mm_D2.5mm_P7.62mm_Horizontal, F.Cu at (118.6, 45.2)
- added R8: 1k, Resistor_THT:R_Axial_DIN0207_L6.3mm_D2.5mm_P7.62mm_Horizontal, F.Cu at (174.0, 118.4)
- added R9: 1k, Resistor_THT:R_Axial_DIN0207_L6.3mm_D2.5mm_P7.62mm_Horizontal, F.Cu at (203.2, 68.8)
- added U20: 74HC688, Package_DIP:DIP-20_W7.62mm_Socket, F.Cu at (165.1, 132.1)
- added U21: 74HC02, Package_DIP:DIP-14_W7.62mm_Socket, F.Cu at (94.0, 133.6)
- added U22: 74HC688, Package_DIP:DIP-20_W7.62mm_Socket, F.Cu at (177.8, 132.1)
- added U23: W65C51NxP, Package_DIP:DIP-28_W15.24mm_Socket, F.Cu at (183.9, 63.8)
- added Y2: 1.8432 MHz, Crystal:Crystal_HC50_Vertical, F.Cu at (178.8, 75.9)
- J1: value BUS -> VIA; footprint edgeconn:DIP-60_200_ELL -> Connector_PinHeader_2.54mm:PinHeader_2x20_P2.54mm_Vertical
- U14: value 74HC193 -> 74HC273; footprint Package_DIP:DIP-16_W7.62mm_Socket -> Package_DIP:DIP-20_W7.62mm_Socket
- U15: value 74HC193 -> 74HC245; footprint Package_DIP:DIP-16_W7.62mm_Socket -> Package_DIP:DIP-20_W7.62mm_Socket
- U8: value CY62256-70PC -> AS6C4008-55PCN; footprint Package_DIP:DIP-28_W15.24mm_Socket -> Package_DIP:DIP-32_W15.24mm
- moved TP2 147.1 mm to (42.2, 154.9)
- moved TP6 102.8 mm to (208.8, 143.8)
- moved TP5 99.9 mm to (208.8, 135.5)
- moved TP4 98.0 mm to (208.8, 127.3)
- moved TP1 91.6 mm to (208.8, 110.9)
- moved TP3 88.6 mm to (208.8, 119.1)
- moved J1 44.4 mm to (165.6, 70.1), turned to 0 degrees
- moved R6 22.9 mm to (83.8, 134.6), turned to 90 degrees
- moved R1 20.1 mm to (42.2, 62.0), turned to -90 degrees
- moved D1 16.0 mm to (76.2, 127.0)
- moved R5 10.4 mm to (96.5, 138.7)
- moved U8 10.2 mm to (66.0, 81.3)
- moved C4 10.0 mm to (84.8, 81.3), turned to -90 degrees
- moved J3 6.92 mm to (166.1, 45.2)
- moved X1 6.86 mm to (26.6, 146.8)
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Connections:
- net ~{IRQC51} renamed ~{IRQC51_1}
- J1 pad 1: A0 -> VCC
- J1 pad 10: A9 -> GND
- J1 pad 11: A10 -> GND
- J1 pad 12: A11 -> PB0
- J1 pad 13: A12 -> PB1
- J1 pad 14: A13 -> PB2
- J1 pad 15: A14 -> PB3
- J1 pad 16: A15 -> PB4
- J1 pad 17: D0 -> PB5
- J1 pad 18: D1 -> PB6
- J1 pad 19: D2 -> PB7
- J1 pad 2: A1 -> PA0
- J1 pad 20: D3 -> GND
- J1 pad 21: D4 -> GND
- J1 pad 22: D5 -> CLK
- J1 pad 23: D6 -> R/~{W}
- J1 pad 24: D7 -> ~{CTS2}
- J1 pad 25: R/~{W} -> RxD2
- J1 pad 26: CLK -> TxD2
- J1 pad 27: ~{RES} -> ~{RTS2}
- J1 pad 28: ~{IRQ} -> ~{CTS1}
- J1 pad 29: ~{I/O} -> RxD1
- J1 pad 3: A2 -> PA1
- J1 pad 30: ~{NMI} -> TxD1
- J1 pad 31: GND -> ~{RTS1}
- J1 pad 32: REG7 -> ~{NMI}
- J1 pad 33: REG6 -> ~{IRQC22}
- J1 pad 34: RAMBANK -> ~{I/O}
- J1 pad 35: BANK4 -> ~{RES}
- J1 pad 36: BANK3 -> CB2
- J1 pad 37: BANK2 -> CB1
- J1 pad 38: BANK1 -> CA2
- J1 pad 39: BANK0 -> CA1
- J1 pad 4: A3 -> PA2
- J1 pad 40: CB2 -> VCC
- J1 pad 5: A4 -> PA3
- J1 pad 6: A5 -> PA4
- J1 pad 7: A6 -> PA5
- J1 pad 8: A7 -> PA6
- J1 pad 9: A8 -> PA7
- J3 pad 1: ~{RTS} -> ~{RTS1}
- J3 pad 2: TxD -> TxD1
- J3 pad 3: RxD -> RxD1
- J3 pad 5: ~{CTS} -> ~{CTS1}
- U11 pad 1: Net-(U8-~{OE}) -> Net-(U8-OE#)
- U14 pad 1: Net-(RN1-R3) -> ~{RES}
- U14 pad 10: Net-(RN1-R2) -> GND
- U14 pad 11: Net-(U14-~{BO}) -> Net-(U14-Cp)
- U14 pad 12: unconnected-(U14-~{CO}-Pad12) -> Net-(U14-Q4)
- U14 pad 13: Net-(U14-~{BO}) -> D4
- U14 pad 14: GND -> D5
- U14 pad 15: Net-(RN1-R4) -> Net-(U14-Q5)
- U14 pad 16: VCC -> Net-(U14-Q6)
- U14 pad 2: unconnected-(U14-QB-Pad2) -> Net-(U14-Q0)
- U14 pad 3: unconnected-(U14-QA-Pad3) -> D0
- U14 pad 4: Net-(U14-DOWN) -> D1
- U14 pad 5: VCC -> Net-(U14-Q1)
- U14 pad 6: unconnected-(U14-QC-Pad6) -> Net-(U14-Q2)
- U14 pad 7: unconnected-(U14-QD-Pad7) -> D2
- U14 pad 8: GND -> D3
- U14 pad 9: Net-(RN1-R1) -> Net-(U14-Q3)
- U15 pad 1: unconnected-(U15-B-Pad1) -> VCC
- U15 pad 10: unconnected-(U15-C-Pad10) -> GND
- U15 pad 11: VCC -> D7
- U15 pad 12: unconnected-(U15-~{CO}-Pad12) -> D6
- U15 pad 13: unconnected-(U15-~{BO}-Pad13) -> D5
- U15 pad 14: GND -> D4
- U15 pad 15: unconnected-(U15-A-Pad15) -> D3
- U15 pad 16: VCC -> D2
- U15 pad 2: unconnected-(U15-QB-Pad2) -> Net-(U14-Q0)
- U15 pad 3: Net-(U15-QA) -> Net-(U14-Q1)
- U15 pad 4: VCC -> Net-(U14-Q2)
- U15 pad 5: Net-(U14-~{BO}) -> Net-(U14-Q3)
- U15 pad 6: unconnected-(U15-QC-Pad6) -> Net-(U14-Q4)
- U15 pad 7: unconnected-(U15-QD-Pad7) -> Net-(U14-Q5)
- U15 pad 8: GND -> Net-(U14-Q6)
- U15 pad 9: unconnected-(U15-D-Pad9) -> Net-(U14-Q7)
- U16 pad 1: Net-(U15-QA) -> Net-(X1-OUT)
- U18 pad 8: Net-(U8-~{CS}) -> Net-(U8-CE#)
- U19 pad 10: GND -> Net-(U19-Pad10)
- U19 pad 11: unconnected-(U19-Pad11) -> Net-(U19-Pad10)
- U19 pad 12: GND -> ~{IRQC51_2}
- U19 pad 13: GND -> VCC
- U19 pad 3: ~{IRQ} -> Net-(U19-Pad3)
- U19 pad 8: unconnected-(U19-Pad8) -> ~{IRQ}
- U19 pad 9: GND -> Net-(U19-Pad3)
- U2 pad 1: BANK4 -> Net-(U2-A18)
- U2 pad 2: BANK2 -> Net-(U2-A16)
- U2 pad 29: BANK0 -> Net-(U2-A14)
- U2 pad 3: BANK1 -> Net-(U2-A15)
- U2 pad 30: BANK3 -> Net-(U2-A17)
- U3 pad 12: BANK4 -> Net-(U2-A18)
- U3 pad 15: RAMBANK -> Net-(U3-Q5)
- U3 pad 16: REG6 -> Net-(U3-Q6)
- U3 pad 19: REG7 -> Net-(U3-Q7)
- U3 pad 2: BANK0 -> Net-(U2-A14)
- U3 pad 5: BANK1 -> Net-(U2-A15)
- U3 pad 6: BANK2 -> Net-(U2-A16)
- U3 pad 9: BANK3 -> Net-(U2-A17)
- U5 pad 10: TxD -> TxD1
- U5 pad 12: RxD -> RxD1
- U5 pad 16: GND -> unconnected-(U5-~{DCD}-Pad16)
- U5 pad 17: GND -> unconnected-(U5-~{DSR}-Pad17)
- U5 pad 8: ~{RTS} -> ~{RTS1}
- U5 pad 9: ~{CTS} -> ~{CTS1}
- U6 pad 4: GND -> Net-(U21-Pad4)
- U6 pad 5: GND -> CLK
- U6 pad 6: unconnected-(U6-Pad6) -> Net-(U14-Cp)
- U8 pad 1: RAMBANK -> Net-(U14-Q4)
- U8 pad 10: A0 -> A2
- U8 pad 11: D0 -> A1
- U8 pad 12: D1 -> A0
- U8 pad 13: D2 -> D0
- U8 pad 14: GND -> D1
- U8 pad 15: D3 -> D2
- U8 pad 16: D4 -> GND
- U8 pad 17: D5 -> D3
- U8 pad 18: D6 -> D4
- U8 pad 19: D7 -> D5
- U8 pad 2: A12 -> Net-(U14-Q2)
- U8 pad 20: Net-(U8-~{CS}) -> D6
- U8 pad 21: A10 -> D7
- U8 pad 22: Net-(U8-~{OE}) -> Net-(U8-CE#)
- U8 pad 23: A11 -> A10
- U8 pad 24: A9 -> Net-(U8-OE#)
- U8 pad 25: A8 -> A11
- U8 pad 26: A13 -> A9
- U8 pad 27: R/~{W} -> A8
- U8 pad 28: VCC -> A13
- U8 pad 3: A7 -> Net-(U14-Q0)
- U8 pad 4: A6 -> A12
- U8 pad 5: A5 -> A7
- U8 pad 6: A4 -> A6
- U8 pad 7: A3 -> A5
- U8 pad 8: A2 -> A4
- U8 pad 9: A1 -> A3
- U9 pad 2: BANK0 -> Net-(U2-A14)
- U9 pad 3: BANK1 -> Net-(U2-A15)
- U9 pad 4: BANK2 -> Net-(U2-A16)
- U9 pad 5: BANK3 -> Net-(U2-A17)
- U9 pad 6: BANK4 -> Net-(U2-A18)
- U9 pad 7: RAMBANK -> Net-(U3-Q5)
- U9 pad 8: REG6 -> Net-(U3-Q6)
- U9 pad 9: REG7 -> Net-(U3-Q7)
- X1 pad 8: Net-(U14-DOWN) -> Net-(X1-OUT)
Routing:
- net GND: track 1688.2 -> 1125.2 mm
- net CLK: track 347.2 -> 0.00 mm, vias 4 -> 0
- net ~{RES}: track 344.8 -> 0.00 mm, vias 2 -> 0
- net ~{NMI}: track 320.7 -> 0.00 mm, vias 8 -> 0
- net A3: track 300.0 -> 0.00 mm, vias 2 -> 0
- net D6: track 297.2 -> 0.00 mm, vias 2 -> 0
- net D3: track 293.7 -> 0.00 mm, vias 1 -> 0
- net D4: track 292.2 -> 0.00 mm, vias 1 -> 0
- net D2: track 291.1 -> 0.00 mm
- net A5: track 290.3 -> 0.00 mm, vias 2 -> 0
- net A7: track 287.3 -> 0.00 mm, vias 1 -> 0
- net A6: track 286.1 -> 0.00 mm
- net A4: track 282.0 -> 0.00 mm, vias 2 -> 0
- net D1: track 275.5 -> 0.00 mm
- net D5: track 275.3 -> 0.00 mm, vias 2 -> 0
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- removed copper zone on In1.Cu, net GND
- removed copper zone on In2.Cu, net VCC
Other:
- board size 157.5 x 119.4 mm -> 191.3 x 119.4 mm
- board text removed: "A0"
- board text removed: "A1"
- board text removed: "A10"
- board text removed: "A11"
- board text removed: "A12"
- board text removed: "A13"
- board text removed: "A14"
- board text removed: "A15"
- board text removed: "A2"
- board text removed: "A3"
- board text removed: "A4"
- board text removed: "A5"
- board text removed: "A6"
- board text removed: "A7"
- board text removed: "A8"
- board text removed: "A9"
- board text removed: "B0"
- board text removed: "B1"
- board text removed: "B2"
- board text removed: "B3"
- board text removed: "B4"
- board text removed: "CA1"
- board text removed: "CA2"
- board text removed: "CB1"
- board text removed: "CB2"
- board text removed: "CLK"
- board text removed: "D0"
- board text removed: "D1"
- board text removed: "D2"
- board text removed: "D3"
- board text removed: "D4"
- board text removed: "D5"
- board text removed: "D6"
- board text removed: "D7"
- board text removed: "PA0"
- board text removed: "PA1"
- board text removed: "PA2"
- board text removed: "PA3"
- board text removed: "PA4"
- board text removed: "PA5"
- board text removed: "PA6"
- board text removed: "PA7"
- board text removed: "PB0"
- board text removed: "PB1"
- board text removed: "PB2"
- board text removed: "PB3"
- board text removed: "PB4"
- board text removed: "PB5"
- board text removed: "PB6"
- board text removed: "PB7"
- board text removed: "R/~{W}"
- board text removed: "R6"
- board text removed: "R7"
- board text removed: "RB"
- board text removed: "~{I/O}"
- board text removed: "~{IRQ}"
- board text removed: "~{NMI}"
- board text removed: "~{RES}"

Commit message: Further redesigning boards
Parts:
- removed C31: 100nF, Capacitor_THT:C_Disc_D5.0mm_W2.5mm_P5.00mm
- added C24: 100nF, Capacitor_THT:C_Disc_D5.0mm_W2.5mm_P5.00mm, F.Cu at (251.5, 81.9)
- added SW1: SW_SPDT, components:power_switch, F.Cu at (69.8, 53.3)
- C1, C29: value 30pF -> 100nF
- C18: value 10uF -> 100nF; footprint Capacitor_THT:CP_Radial_D6.3mm_P2.50mm -> Capacitor_THT:C_Disc_D5.0mm_W2.5mm_P5.00mm
- C19: value 100uF -> 100nF; footprint Capacitor_THT:CP_Radial_D6.3mm_P2.50mm -> Capacitor_THT:C_Disc_D5.0mm_W2.5mm_P5.00mm
- C25, C28: value 100nF -> 30pF
- C6: value 100nF -> 10uF; footprint Capacitor_THT:C_Disc_D5.0mm_W2.5mm_P5.00mm -> Capacitor_THT:CP_Radial_D6.3mm_P2.50mm
- C7: value 100nF -> 100uF; footprint Capacitor_THT:C_Disc_D5.0mm_W2.5mm_P5.00mm -> Capacitor_THT:CP_Radial_D6.3mm_P2.50mm
- J1: value VIA -> USB_B; footprint Connector_PinHeader_2.54mm:PinHeader_2x20_P2.54mm_Vertical -> Connector_USB:USB_B_OST_USB-B1HSxx_Horizontal
- J2: value USB_B -> EXPBUS1; footprint Connector_USB:USB_B_OST_USB-B1HSxx_Horizontal -> Connector_PinHeader_2.54mm:PinHeader_2x20_P2.54mm_Vertical
- J3: value Serial -> EXPBUS2; footprint Connector_PinSocket_2.54mm:PinSocket_1x06_P2.54mm_Vertical -> Connector_PinHeader_2.54mm:PinHeader_2x20_P2.54mm_Vertical
- J4: value Serial -> VIA; footprint Connector_PinSocket_2.54mm:PinSocket_1x06_P2.54mm_Vertical -> Connector_PinHeader_2.54mm:PinHeader_2x20_P2.54mm_Vertical
- J5: value EXPBUS1 -> UART1; footprint Connector_PinHeader_2.54mm:PinHeader_2x20_P2.54mm_Vertical -> Connector_Dsub:DSUB-9_Male_Horizontal_P2.77x2.84mm_EdgePinOffset4.94mm_Housed_MountingHolesOffset7.48mm
- J6: value EXPBUS2 -> UART2; footprint Connector_PinHeader_2.54mm:PinHeader_2x20_P2.54mm_Vertical -> Connector_Dsub:DSUB-9_Male_Horizontal_P2.77x2.84mm_EdgePinOffset4.94mm_Housed_MountingHolesOffset7.48mm
- J7: value UART1 -> Serial; footprint Connector_Dsub:DSUB-9_Male_Horizontal_P2.77x2.84mm_EdgePinOffset4.94mm_Housed_MountingHolesOffset7.48mm -> Connector_PinSocket_2.54mm:PinSocket_1x06_P2.54mm_Vertical
- J8: value UART2 -> Serial; footprint Connector_Dsub:DSUB-9_Male_Horizontal_P2.77x2.84mm_EdgePinOffset4.94mm_Housed_MountingHolesOffset7.48mm -> Connector_PinSocket_2.54mm:PinSocket_1x06_P2.54mm_Vertical
- R2: value 1k -> 100k
- R3: value 1M -> 560
- R4: value 100k -> 1k
- R6: value 560 -> 1k
- R8: value 1k -> 1M
- U1: value W65C02SxP -> 74HC14; footprint Package_DIP:DIP-40_W15.24mm_Socket -> Package_DIP:DIP-14_W7.62mm_Socket
- U10: value 74HC688 -> 74HC00; footprint Package_DIP:DIP-20_W7.62mm_Socket -> Package_DIP:DIP-14_W7.62mm_Socket
- U11: value 74HC02 -> 74HC273; footprint Package_DIP:DIP-14_W7.62mm_Socket -> Package_DIP:DIP-20_W7.62mm_Socket
- U12: value 74HC688 -> 74HC273
- U13: value W65C22NxP -> 74HC245; footprint Package_DIP:DIP-40_W15.24mm_Socket -> Package_DIP:DIP-20_W7.62mm_Socket
- U14: value 74HC273 -> 74HC245
- U15: value 74HC245 -> SST39SF040; footprint Package_DIP:DIP-20_W7.62mm_Socket -> Socket:DIP_Socket-32_W11.9_W12.7_W15.24_W17.78_W18.5_3M_232-1285-00-0602J
- U16: value 74HC14 -> AS6C4008; footprint Package_DIP:DIP-14_W7.62mm_Socket -> Package_DIP:DIP-32_W15.24mm
- U17: value 74HC688 -> CY62256; footprint Package_DIP:DIP-20_W7.62mm_Socket -> Package_DIP:DIP-28_W15.24mm_Socket
- U18, U6: value 74HC00 -> 74HC688; footprint Package_DIP:DIP-14_W7.62mm_Socket -> Package_DIP:DIP-20_W7.62mm_Socket
- U19: value 74HC08 -> W65C22NxP; footprint Package_DIP:DIP-14_W7.62mm_Socket -> Package_DIP:DIP-40_W15.24mm_Socket
- U2: value SST39SF040 -> W65C02; footprint Socket:DIP_Socket-32_W11.9_W12.7_W15.24_W17.78_W18.5_3M_232-1285-00-0602J -> Package_DIP:DIP-40_W15.24mm_Socket
- U21: value 74HC02 -> W65C51NxP; footprint Package_DIP:DIP-14_W7.62mm_Socket -> Package_DIP:DIP-28_W15.24mm_Socket
- U3: value 74HC273 -> 74HC688
- U4: value 74HC688 -> 74HC08; footprint Package_DIP:DIP-20_W7.62mm_Socket -> Package_DIP:DIP-14_W7.62mm_Socket
- U5: value W65C51NxP -> 74HC688; footprint Package_DIP:DIP-28_W15.24mm_Socket -> Package_DIP:DIP-20_W7.62mm_Socket
- U7: value CY62256-70PC -> 74HC02; footprint Package_DIP:DIP-28_W15.24mm_Socket -> Package_DIP:DIP-14_W7.62mm_Socket
- U8: value AS6C4008-55PCN -> 74HC02; footprint Package_DIP:DIP-32_W15.24mm -> Package_DIP:DIP-14_W7.62mm_Socket
- U9: value 74HC245 -> 74HC00; footprint Package_DIP:DIP-20_W7.62mm_Socket -> Package_DIP:DIP-14_W7.62mm_Socket
- moved U19 197.9 mm to (241.3, 87.0)
- moved J2 184.2 mm to (215.9, 59.7)
- moved R6 177.9 mm to (261.6, 127.6), turned to -90 degrees
- moved C18 167.2 mm to (182.9, 127.0), turned to -90 degrees
- moved U15 158.8 mm to (215.3, 94.6)
- moved U18 155.0 mm to (241.3, 73.7)
- moved C23 151.5 mm to (236.2, 67.3), turned to -90 degrees
- moved C19 151.4 mm to (182.9, 114.3), turned to -90 degrees
- moved U7 142.6 mm to (188.0, 95.2), turned to 90 degrees
- moved C16 137.1 mm to (225.4, 80.0), turned to 180 degrees
- moved U10 130.6 mm to (188.0, 108.0), turned to 90 degrees
- moved U8 128.1 mm to (188.0, 120.7), turned to 90 degrees
- moved C2 118.2 mm to (147.3, 88.9), turned to -90 degrees
- moved C27 112.5 mm to (86.4, 53.4), turned to -90 degrees
- moved TP1 110.5 mm to (101.6, 137.8)
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Connections:
- C1 pad 1: GND -> VCC
- C1 pad 2: Net-(U5-XTAL1) -> GND
- C22 pad 1: ~{RES} -> VCC
- C23 pad 1: ~{NMI} -> VCC
- C25 pad 1: VCC -> GND
- C25 pad 2: GND -> Net-(U21-XTAL1)
- C28 pad 1: VCC -> GND
- C28 pad 2: GND -> Net-(U23-XTAL1)
- C29 pad 1: GND -> VCC
- C29 pad 2: Net-(U23-XTAL1) -> GND
- C8 pad 1: VCC -> ~{RES}
- C9 pad 1: VCC -> ~{NMI}
- J1 pad 1: VCC -> VIN
- J1 pad 2: PA0 -> unconnected-(J1-D--Pad2)
- J1 pad 3: PA1 -> unconnected-(J1-D+-Pad3)
- J1 pad 4: PA2 -> GND
- J1 pad 5: PA3 -> Net-(J1-Shield)
- J2 pad 2: unconnected-(J2-D--Pad2) -> VCC
- J2 pad 3: unconnected-(J2-D+-Pad3) -> A0
- J2 pad 4: GND -> R/~{W}
- J2 pad 5: Net-(J2-Shield) -> A1
- J3 pad 1: ~{RTS1} -> VCC
- J3 pad 2: TxD1 -> VCC
- J3 pad 3: RxD1 -> A0
- J3 pad 4: VCC -> R/~{W}
- J3 pad 5: ~{CTS1} -> A1
- J3 pad 6: GND -> CLK
- J4 pad 1: ~{RTS2} -> VCC
- J4 pad 2: TxD2 -> VCC
- J4 pad 3: RxD2 -> PA0
- J4 pad 4: VCC -> CA1
- J4 pad 5: ~{CTS2} -> PA1
- J4 pad 6: GND -> CA2
- J5 pad 1: VCC -> unconnected-(J5-Pad1)
- J5 pad 2: A0 -> TxD1
- J5 pad 3: A1 -> RxD1
- J5 pad 4: A2 -> unconnected-(J5-Pad4)
- J5 pad 5: A3 -> GND
- J5 pad 6: A4 -> unconnected-(J5-Pad6)
- J5 pad 7: A5 -> ~{CTS1}
- J5 pad 8: A6 -> ~{RTS1}
- J5 pad 9: A7 -> unconnected-(J5-Pad9)
- J6 pad 1: VCC -> unconnected-(J6-Pad1)
- J6 pad 2: A0 -> TxD2
- J6 pad 3: A1 -> RxD2
- J6 pad 4: A2 -> unconnected-(J6-Pad4)
- J6 pad 5: A3 -> GND
- J6 pad 6: A4 -> unconnected-(J6-Pad6)
- J6 pad 7: A5 -> ~{CTS2}
- J6 pad 8: A6 -> ~{RTS2}
- J6 pad 9: A7 -> unconnected-(J6-Pad9)
- J7 pad 1: unconnected-(J7-Pad1) -> ~{RTS1}
- J7 pad 4: unconnected-(J7-Pad4) -> VCC
- J7 pad 5: GND -> ~{CTS1}
- J7 pad 6: unconnected-(J7-Pad6) -> GND
- J8 pad 1: unconnected-(J8-Pad1) -> ~{RTS2}
- J8 pad 4: unconnected-(J8-Pad4) -> VCC
- J8 pad 5: GND -> ~{CTS2}
- J8 pad 6: unconnected-(J8-Pad6) -> GND
- R1 pad 2: Net-(U1-RDY) -> Net-(U2-RDY)
- R2 pad 1: ~{IRQC51_1} -> GND
- R2 pad 2: VCC -> Net-(J1-Shield)
- R3 pad 1: Net-(U5-XTAL1) -> GND
- R3 pad 2: Net-(U5-XTAL2) -> Net-(D1-K)
- R4 pad 1: GND -> ~{RES}
- R4 pad 2: Net-(J2-Shield) -> VCC
- R5 pad 1: ~{RES} -> ~{NMI}
- R6 pad 1: GND -> VCC
- R6 pad 2: Net-(D1-K) -> ~{IRQC22}
- R7 pad 1: ~{NMI} -> ~{IRQC51_1}
- R8 pad 1: VCC -> Net-(U21-XTAL1)
- R8 pad 2: ~{IRQC22} -> Net-(U21-XTAL2)
- U1 pad 1: unconnected-(U1-~{VP}-Pad1) -> Net-(X1-OUT)
- U1 pad 10: A1 -> unconnected-(U1-Pad10)
- U1 pad 11: A2 -> GND
- U1 pad 12: A3 -> unconnected-(U1-Pad12)
- U1 pad 13: A4 -> GND
- U1 pad 14: A5 -> VCC
- U1 pad 2: Net-(U1-RDY) -> Net-(U1-Pad2)
- U1 pad 3: unconnected-(U1-ϕ1-Pad3) -> Net-(U1-Pad2)
- U1 pad 4: ~{IRQ} -> CLK
- U1 pad 5: unconnected-(U1-~{ML}-Pad5) -> CLK
- U1 pad 6: ~{NMI} -> ~{CLK}
- U1 pad 7: unconnected-(U1-SYNC-Pad7) -> GND
- U1 pad 8: VCC -> unconnected-(U1-Pad8)
- U1 pad 9: A0 -> GND
- U10 pad 1: ~{I/O} -> Net-(U10-Pad1)
- U10 pad 10: GND -> Net-(U10-Pad10)
- U10 pad 11: A4 -> Net-(U10-Pad10)
- U10 pad 12: GND -> ~{I/O}
- U10 pad 13: A5 -> Net-(U10-Pad13)
- U10 pad 14: GND -> VCC
- U10 pad 2: A0 -> R/~{W}
- U10 pad 3: GND -> Net-(U14-CE)
- U10 pad 4: A1 -> Net-(U10-Pad4)
- U10 pad 5: GND -> CLK
- U10 pad 6: A2 -> Net-(U12-Cp)
- U10 pad 8: A3 -> Net-(U17-~{CS})
- U10 pad 9: GND -> CLK
- U11 pad 1: Net-(U8-OE#) -> ~{RES}
- U11 pad 10: Net-(U11-Pad10) -> GND
- U11 pad 11: Net-(U10-P=R) -> Net-(U11-Cp)
- U11 pad 12: Net-(U10-P=R) -> Net-(U11-Q4)
- U11 pad 13: Net-(U11-Pad13) -> D4
- U11 pad 14: VCC -> D5
- U11 pad 2: Net-(U11-Pad2) -> Net-(U11-Q0)
- U11 pad 3: Net-(U11-Pad2) -> D0
- U11 pad 4: Net-(U11-Pad2) -> D1
- U11 pad 5: Net-(U11-Pad5) -> Net-(U11-Q1)
- U11 pad 6: A14 -> Net-(U11-Q2)
- U11 pad 7: GND -> D2
- U11 pad 8: R/~{W} -> D3
- U11 pad 9: Net-(U10-P=R) -> Net-(U11-Q3)
- U12 pad 1: ~{I/O} -> ~{RES}
- U12 pad 11: A4 -> Net-(U12-Cp)
- U12 pad 12: GND -> Net-(U12-Q4)
- U12 pad 13: A5 -> D4
- U12 pad 14: GND -> D5
- U12 pad 15: A6 -> Net-(U12-Q5)
- U12 pad 16: GND -> Net-(U12-Q6)
- U12 pad 17: A7 -> D6
- U12 pad 18: GND -> D7
- U12 pad 19: Net-(U12-P=R) -> Net-(U12-Q7)
- U12 pad 2: GND -> Net-(U12-Q0)
- U12 pad 3: GND -> D0
- U12 pad 4: GND -> D1
- U12 pad 5: GND -> Net-(U12-Q1)
- U12 pad 6: A2 -> Net-(U12-Q2)
- U12 pad 7: VCC -> D2
- U12 pad 8: A3 -> D3
- U12 pad 9: GND -> Net-(U12-Q3)
- U13 pad 1: GND -> VCC
- U13 pad 10: PB0 -> GND
- U13 pad 11: PB1 -> D7
- U13 pad 12: PB2 -> D6
- U13 pad 13: PB3 -> D5
- U13 pad 14: PB4 -> D4
- U13 pad 15: PB5 -> D3
- U13 pad 16: PB6 -> D2
- U13 pad 17: PB7 -> D1
- U13 pad 18: CB1 -> D0
- U13 pad 19: CB2 -> Net-(U13-CE)
- U13 pad 2: PA0 -> Net-(U11-Q0)
- U13 pad 3: PA1 -> Net-(U11-Q1)
- U13 pad 4: PA2 -> Net-(U11-Q2)
- U13 pad 5: PA3 -> Net-(U11-Q3)
- U13 pad 6: PA4 -> Net-(U11-Q4)
- U13 pad 7: PA5 -> Net-(U11-Q5)
- U13 pad 8: PA6 -> Net-(U11-Q6)
- U13 pad 9: PA7 -> Net-(U11-Q7)
- U14 pad 1: ~{RES} -> VCC
- U14 pad 11: Net-(U14-Cp) -> D7
- U14 pad 12: Net-(U14-Q4) -> D6
- U14 pad 13: D4 -> D5
- U14 pad 14: D5 -> D4
- U14 pad 15: Net-(U14-Q5) -> D3
- U14 pad 16: Net-(U14-Q6) -> D2
- U14 pad 17: D6 -> D1
- U14 pad 18: D7 -> D0
- U14 pad 19: Net-(U14-Q7) -> Net-(U14-CE)
- U14 pad 2: Net-(U14-Q0) -> Net-(U12-Q0)
- U14 pad 3: D0 -> Net-(U12-Q1)
- U14 pad 4: D1 -> Net-(U12-Q2)
- U14 pad 5: Net-(U14-Q1) -> Net-(U12-Q3)
- U14 pad 6: Net-(U14-Q2) -> Net-(U12-Q4)
- U14 pad 7: D2 -> Net-(U12-Q5)
- U14 pad 8: D3 -> Net-(U12-Q6)
- U14 pad 9: Net-(U14-Q3) -> Net-(U12-Q7)
- U15 pad 1: VCC -> Net-(U11-Q4)
- U15 pad 10: GND -> A2
- U15 pad 11: D7 -> A1
- U15 pad 12: D6 -> A0
- U15 pad 13: D5 -> D0
- U15 pad 14: D4 -> D1
- U15 pad 15: D3 -> D2
- U15 pad 16: D2 -> GND
- U15 pad 17: D1 -> D3
- U15 pad 18: D0 -> D4
- U15 pad 19: Net-(U15-CE) -> D5
- U15 pad 2: Net-(U14-Q0) -> Net-(U11-Q2)
- U15 pad 20: VCC -> D6
- U15 pad 3: Net-(U14-Q1) -> Net-(U11-Q1)
- U15 pad 4: Net-(U14-Q2) -> A12
- U15 pad 5: Net-(U14-Q3) -> A7
- U15 pad 6: Net-(U14-Q4) -> A6
- U15 pad 7: Net-(U14-Q5) -> A5
- U15 pad 8: Net-(U14-Q6) -> A4
- U15 pad 9: Net-(U14-Q7) -> A3
- U16 pad 1: Net-(X1-OUT) -> Net-(U12-Q4)
- U16 pad 10: unconnected-(U16-Pad10) -> A2
- U16 pad 11: GND -> A1
- U16 pad 12: unconnected-(U16-Pad12) -> A0
- U16 pad 13: GND -> D0
- U16 pad 14: VCC -> D1
- U16 pad 2: Net-(U16-Pad2) -> Net-(U12-Q2)
- U16 pad 3: Net-(U16-Pad2) -> Net-(U12-Q0)
- U16 pad 4: CLK -> A12
- U16 pad 5: CLK -> A7
- U16 pad 6: ~{CLK} -> A6
- U16 pad 7: GND -> A5
- U16 pad 8: unconnected-(U16-Pad8) -> A4
- U16 pad 9: GND -> A3
- U17 pad 1: ~{I/O} -> A14
- U17 pad 10: GND -> A0
- U17 pad 11: A4 -> D0
- U17 pad 12: VCC -> D1
- U17 pad 13: A5 -> D2
- U17 pad 15: A6 -> D3
- U17 pad 16: GND -> D4
- U17 pad 17: A7 -> D5
- U17 pad 18: GND -> D6
- U17 pad 19: Net-(U13-~{CS2}) -> D7
- U17 pad 2: GND -> A12
- U17 pad 20: VCC -> Net-(U17-~{CS})
- U17 pad 3: GND -> A7
- U17 pad 4: GND -> A6
- U17 pad 5: GND -> A5
- U17 pad 6: GND -> A4
- U17 pad 7: GND -> A3
- U17 pad 8: GND -> A2
- U17 pad 9: GND -> A1
- U18 pad 1: Net-(U11-Pad10) -> ~{I/O}
- U18 pad 10: CLK -> GND
- U18 pad 11: Net-(U7-~{CS}) -> A4
- U18 pad 12: Net-(U18-Pad12) -> VCC
- U18 pad 13: CLK -> A5
- U18 pad 14: VCC -> GND
- U18 pad 2: CLK -> GND
- U18 pad 3: Net-(U3-Cp) -> GND
- U18 pad 4: Net-(U11-Pad13) -> GND
- U18 pad 5: R/~{W} -> GND
- U18 pad 6: Net-(U9-CE) -> GND
- U18 pad 8: Net-(U8-CE#) -> GND
- U18 pad 9: Net-(U11-Pad2) -> GND
- U19 pad 1: ~{IRQC22} -> GND
- U19 pad 10: Net-(U19-Pad10) -> PB0
- U19 pad 11: Net-(U19-Pad10) -> PB1
- U19 pad 12: ~{IRQC51_2} -> PB2
- U19 pad 13: VCC -> PB3
- U19 pad 14: VCC -> PB4
- U19 pad 2: ~{IRQC51_1} -> PA0
- U19 pad 3: Net-(U19-Pad3) -> PA1
- U19 pad 4: GND -> PA2
- U19 pad 5: GND -> PA3
- U19 pad 6: unconnected-(U19-Pad6) -> PA4
- U19 pad 7: GND -> PA5
- U19 pad 8: ~{IRQ} -> PA6
- U19 pad 9: Net-(U19-Pad3) -> PA7
- U2 pad 1: Net-(U2-A18) -> unconnected-(U2-~{VP}-Pad1)
- U2 pad 10: A2 -> A1
- U2 pad 11: A1 -> A2
- U2 pad 12: A0 -> A3
- U2 pad 13: D0 -> A4
- U2 pad 14: D1 -> A5
- U2 pad 15: D2 -> A6
- U2 pad 16: GND -> A7
- U2 pad 17: D3 -> A8
- U2 pad 18: D4 -> A9
- U2 pad 19: D5 -> A10
- U2 pad 2: Net-(U2-A16) -> Net-(U2-RDY)
- U2 pad 20: D6 -> A11
- U2 pad 21: D7 -> GND
- U2 pad 22: Net-(U2-CE) -> A12
- U2 pad 23: A10 -> A13
- U2 pad 24: Net-(U2-CE) -> A14
- U2 pad 25: A11 -> A15
- U2 pad 26: A9 -> D7
- U2 pad 27: A8 -> D6
- U2 pad 28: A13 -> D5
- U2 pad 29: Net-(U2-A14) -> D4
- U2 pad 3: Net-(U2-A15) -> unconnected-(U2-ϕ1-Pad3)
- U2 pad 30: Net-(U2-A17) -> D3
- U2 pad 31: VCC -> D2
- U2 pad 32: VCC -> D1
- U2 pad 4: A12 -> ~{IRQ}
- U2 pad 5: A7 -> unconnected-(U2-~{ML}-Pad5)
- U2 pad 6: A6 -> ~{NMI}
- U2 pad 7: A5 -> unconnected-(U2-SYNC-Pad7)
- U2 pad 8: A4 -> VCC
- U2 pad 9: A3 -> A0
- U20 pad 2: A0 -> GND
- U20 pad 3: VCC -> GND
- U20 pad 4: A1 -> GND
- U20 pad 7: GND -> VCC
- U21 pad 1: Net-(U21-Pad1) -> GND
- U21 pad 10: Net-(U21-Pad10) -> TxD1
- U21 pad 11: Net-(U21-Pad10) -> unconnected-(U21-~{DTR}-Pad11)
- U21 pad 12: Net-(U21-Pad10) -> RxD1
- U21 pad 13: Net-(U15-CE) -> A0
- U21 pad 14: VCC -> A1
- U21 pad 2: R/~{W} -> VCC
- U21 pad 3: R/~{W} -> Net-(U20-P=R)
- U21 pad 4: Net-(U21-Pad4) -> ~{RES}
- U21 pad 5: R/~{W} -> unconnected-(U21-RxC-Pad5)
- U21 pad 6: Net-(U20-P=R) -> Net-(U21-XTAL1)
- U21 pad 7: GND -> Net-(U21-XTAL2)
- U21 pad 8: Net-(U21-Pad1) -> ~{RTS1}
- U21 pad 9: Net-(U20-P=R) -> ~{CTS1}
- U3 pad 1: ~{RES} -> GND
- U3 pad 11: Net-(U3-Cp) -> A12
- U3 pad 12: Net-(U2-A18) -> VCC
- U3 pad 13: D4 -> A13
- U3 pad 14: D5 -> VCC
- U3 pad 15: Net-(U3-Q5) -> A14
- U3 pad 16: Net-(U3-Q6) -> VCC
- U3 pad 17: D6 -> A15
- U3 pad 18: D7 -> GND
- U3 pad 19: Net-(U3-Q7) -> ~{I/O}
- U3 pad 2: Net-(U2-A14) -> A8
- U3 pad 3: D0 -> VCC
- U3 pad 4: D1 -> A9
- U3 pad 5: Net-(U2-A15) -> VCC
- U3 pad 6: Net-(U2-A16) -> A10
- U3 pad 7: D2 -> VCC
- U3 pad 8: D3 -> A11
- U3 pad 9: Net-(U2-A17) -> VCC
- U4 pad 1: GND -> ~{IRQC22}
- U4 pad 10: GND -> Net-(U4-Pad10)
- U4 pad 11: A12 -> Net-(U4-Pad10)
- U4 pad 12: VCC -> ~{IRQC51_2}
- U4 pad 13: A13 -> VCC
- U4 pad 14: GND -> VCC
- U4 pad 2: A8 -> ~{IRQC51_1}
- U4 pad 3: VCC -> Net-(U4-Pad3)
- U4 pad 4: A9 -> GND
- U4 pad 5: VCC -> GND
- U4 pad 6: A10 -> unconnected-(U4-Pad6)
- U4 pad 7: VCC -> GND
- U4 pad 8: A11 -> ~{IRQ}
- U4 pad 9: VCC -> Net-(U4-Pad3)
- U5 pad 1: GND -> ~{I/O}
- U5 pad 10: TxD1 -> GND
- U5 pad 11: unconnected-(U5-~{DTR}-Pad11) -> A4
- U5 pad 12: RxD1 -> GND
- U5 pad 13: A0 -> A5
- U5 pad 14: A1 -> GND
- U5 pad 15: VCC -> A6
- U5 pad 16: unconnected-(U5-~{DCD}-Pad16) -> GND
- U5 pad 17: unconnected-(U5-~{DSR}-Pad17) -> A7
- U5 pad 18: D0 -> GND
- U5 pad 19: D1 -> Net-(U5-P=R)
- U5 pad 2: VCC -> A0
- U5 pad 20: D2 -> VCC
- U5 pad 3: Net-(U12-P=R) -> VCC
- U5 pad 4: ~{RES} -> A1
- U5 pad 5: unconnected-(U5-RxC-Pad5) -> GND
- U5 pad 6: Net-(U5-XTAL1) -> A2
- U5 pad 7: Net-(U5-XTAL2) -> GND
- U5 pad 8: ~{RTS1} -> A3
- U5 pad 9: ~{CTS1} -> GND
- U6 pad 1: A14 -> ~{I/O}
- U6 pad 10: ~{I/O} -> GND
- U6 pad 11: Net-(U18-Pad12) -> A4
- U6 pad 12: A15 -> GND
- U6 pad 13: A15 -> A5
- U6 pad 14: VCC -> GND
- U6 pad 2: A15 -> A0
- U6 pad 3: Net-(U2-CE) -> GND
- U6 pad 4: Net-(U21-Pad4) -> A1
- U6 pad 5: CLK -> GND
- U6 pad 6: Net-(U14-Cp) -> A2
- U6 pad 8: Net-(U11-Pad5) -> A3
- U6 pad 9: A15 -> GND
- U7 pad 1: A14 -> Net-(U15-CE)
- U7 pad 10: A0 -> Net-(U10-Pad1)
- U7 pad 11: D0 -> A15
- U7 pad 12: D1 -> A15
- U7 pad 13: D2 -> Net-(U10-Pad13)
- U7 pad 14: GND -> VCC
- U7 pad 2: A12 -> A14
- U7 pad 3: A7 -> A15
- U7 pad 4: A6 -> Net-(U10-Pad4)
- U7 pad 5: A5 -> R/~{W}
- U7 pad 6: A4 -> Net-(U5-P=R)
- U7 pad 7: A3 -> GND
- U7 pad 8: A2 -> Net-(U5-P=R)
- U7 pad 9: A1 -> Net-(U5-P=R)
- U8 pad 1: Net-(U14-Q4) -> Net-(U8-Pad1)
- U8 pad 10: A2 -> Net-(U8-Pad10)
- U8 pad 11: A1 -> Net-(U6-P=R)
- U8 pad 12: A0 -> Net-(U6-P=R)
- U8 pad 13: D0 -> Net-(U8-Pad13)
- U8 pad 14: D1 -> VCC
- U8 pad 2: Net-(U14-Q2) -> A14
- U8 pad 3: Net-(U14-Q0) -> A14
- U8 pad 4: A12 -> Net-(U8-Pad4)
- U8 pad 5: A7 -> Net-(U16-OE#)
- U8 pad 6: A6 -> Net-(U16-OE#)
- U8 pad 7: A5 -> GND
- U8 pad 8: A4 -> R/~{W}
- U8 pad 9: A3 -> Net-(U6-P=R)
- U9 pad 1: VCC -> Net-(U8-Pad10)
- U9 pad 10: GND -> CLK
- U9 pad 11: D7 -> Net-(U16-OE#)
- U9 pad 12: D6 -> Net-(U8-Pad1)
- U9 pad 13: D5 -> A15
- U9 pad 14: D4 -> VCC
- U9 pad 2: Net-(U2-A14) -> CLK
- U9 pad 3: Net-(U2-A15) -> Net-(U11-Cp)
- U9 pad 4: Net-(U2-A16) -> Net-(U8-Pad13)
- U9 pad 5: Net-(U2-A17) -> R/~{W}
- U9 pad 6: Net-(U2-A18) -> Net-(U13-CE)
- U9 pad 7: Net-(U3-Q5) -> GND
- U9 pad 8: Net-(U3-Q6) -> Net-(U16-CE#)
- U9 pad 9: Net-(U3-Q7) -> Net-(U8-Pad4)
- Y1 pad 1: Net-(U5-XTAL2) -> Net-(U21-XTAL2)
- Y1 pad 2: Net-(U5-XTAL1) -> Net-(U21-XTAL1)
Routing:
- net GND: track 1125.2 -> 1823.6 mm, vias 0 -> 8
- net CLK: track 0.00 -> 509.8 mm, vias 0 -> 4
- net VCC: track 1045.8 -> 1380.6 mm, vias 1 -> 4
- net RxD1: track 0.00 -> 72.0 mm
- net RxD2: track 0.00 -> 70.3 mm
- net ~{RTS1}: track 0.00 -> 65.6 mm
- net ~{RTS2}: track 0.00 -> 65.6 mm
- net ~{CTS1}: track 0.00 -> 62.2 mm, vias 0 -> 2
- net ~{CTS2}: track 0.00 -> 62.2 mm, vias 0 -> 2
- net TxD1: track 0.00 -> 59.9 mm
- net TxD2: track 0.00 -> 59.9 mm
- net Net-(U21-XTAL1): track 0.00 -> 32.0 mm
- net Net-(U23-XTAL1): track 0.00 -> 31.9 mm
- net Net-(J1-Shield): track 0.00 -> 25.7 mm
- net Net-(X1-OUT): track 0.00 -> 22.0 mm
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Other:
- board size 191.3 x 119.4 mm -> 224.9 x 116.2 mm
- copper layers 4 -> 2
- board text added: "OFF"
- board text added: "ON"

Commit message: Fixing mistake
Parts:
- U10: value 74HC00 -> 74HC273; footprint Package_DIP:DIP-14_W7.62mm_Socket -> Package_DIP:DIP-20_W7.62mm_Socket
- U12: value 74HC273 -> 74HC245
- U14: value 74HC245 -> 74HC10; footprint Package_DIP:DIP-20_W7.62mm_Socket -> Package_DIP:DIP-14_W7.62mm_Socket
- U7: value 74HC02 -> 74HC04
- U8: value 74HC02 -> 74HC10
- moved U10 131.0 mm to (57.1, 114.9)
- moved U14 131.0 mm to (188.0, 108.0)
Connections:
- U10 pad 1: Net-(U10-Pad1) -> ~{RES}
- U10 pad 10: Net-(U10-Pad10) -> GND
- U10 pad 11: Net-(U10-Pad10) -> Net-(U10-Cp)
- U10 pad 12: ~{I/O} -> Net-(U10-Q4)
- U10 pad 13: Net-(U10-Pad13) -> D4
- U10 pad 14: VCC -> D5
- U10 pad 2: R/~{W} -> Net-(U10-Q0)
- U10 pad 3: Net-(U14-CE) -> D0
- U10 pad 4: Net-(U10-Pad4) -> D1
- U10 pad 5: CLK -> Net-(U10-Q1)
- U10 pad 6: Net-(U12-Cp) -> Net-(U10-Q2)
- U10 pad 7: GND -> D2
- U10 pad 8: Net-(U17-~{CS}) -> D3
- U10 pad 9: CLK -> Net-(U10-Q3)
- U12 pad 1: ~{RES} -> VCC
- U12 pad 11: Net-(U12-Cp) -> D7
- U12 pad 12: Net-(U12-Q4) -> D6
- U12 pad 13: D4 -> D5
- U12 pad 14: D5 -> D4
- U12 pad 15: Net-(U12-Q5) -> D3
- U12 pad 16: Net-(U12-Q6) -> D2
- U12 pad 17: D6 -> D1
- U12 pad 18: D7 -> D0
- U12 pad 19: Net-(U12-Q7) -> Net-(U12-CE)
- U12 pad 2: Net-(U12-Q0) -> Net-(U10-Q0)
- U12 pad 3: D0 -> Net-(U10-Q1)
- U12 pad 4: D1 -> Net-(U10-Q2)
- U12 pad 5: Net-(U12-Q1) -> Net-(U10-Q3)
- U12 pad 6: Net-(U12-Q2) -> Net-(U10-Q4)
- U12 pad 7: D2 -> Net-(U10-Q5)
- U12 pad 8: D3 -> Net-(U10-Q6)
- U12 pad 9: Net-(U12-Q3) -> Net-(U10-Q7)
- U14 pad 10: GND -> ~{A15}
- U14 pad 11: D7 -> VCC
- U14 pad 12: D6 -> Net-(U15-CE)
- U14 pad 13: D5 -> A15
- U14 pad 14: D4 -> VCC
- U14 pad 2: Net-(U12-Q0) -> A14
- U14 pad 3: Net-(U12-Q1) -> ~{I/O}
- U14 pad 4: Net-(U12-Q2) -> ~{A15}
- U14 pad 5: Net-(U12-Q3) -> CLK
- U14 pad 6: Net-(U12-Q4) -> Net-(U17-~{CS})
- U14 pad 7: Net-(U12-Q5) -> GND
- U14 pad 8: Net-(U12-Q6) -> Net-(U16-OE#)
- U14 pad 9: Net-(U12-Q7) -> ~{A14}
- U15 pad 1: Net-(U11-Q4) -> Net-(U10-Q4)
- U15 pad 2: Net-(U11-Q2) -> Net-(U10-Q2)
- U15 pad 29: Net-(U11-Q0) -> Net-(U10-Q0)
- U15 pad 3: Net-(U11-Q1) -> Net-(U10-Q1)
- U15 pad 30: Net-(U11-Q3) -> Net-(U10-Q3)
- U16 pad 1: Net-(U12-Q4) -> Net-(U11-Q4)
- U16 pad 2: Net-(U12-Q2) -> Net-(U11-Q2)
- U16 pad 3: Net-(U12-Q0) -> Net-(U11-Q0)
- U16 pad 30: Net-(U12-Q3) -> Net-(U11-Q3)
- U16 pad 31: Net-(U12-Q1) -> Net-(U11-Q1)
- U7 pad 1: Net-(U15-CE) -> A15
- U7 pad 10: Net-(U10-Pad1) -> ~{R}/W
- U7 pad 11: A15 -> R/~{W}
- U7 pad 12: A15 -> unconnected-(U7-Pad12)
- U7 pad 13: Net-(U10-Pad13) -> GND
- U7 pad 2: A14 -> ~{A15}
- U7 pad 3: A15 -> A14
- U7 pad 4: Net-(U10-Pad4) -> ~{A14}
- U7 pad 5: R/~{W} -> Net-(U6-P=R)
- U7 pad 6: Net-(U5-P=R) -> Net-(U7-Pad6)
- U7 pad 8: Net-(U5-P=R) -> Net-(U7-Pad8)
- U8 pad 1: Net-(U8-Pad1) -> ~{R}/W
- U8 pad 10: Net-(U8-Pad10) -> ~{R}/W
- U8 pad 11: Net-(U6-P=R) -> Net-(U7-Pad6)
- U8 pad 12: Net-(U6-P=R) -> Net-(U11-Cp)
- U8 pad 13: Net-(U8-Pad13) -> Net-(U7-Pad8)
- U8 pad 14: VCC -> GND
- U8 pad 2: A14 -> CLK
- U8 pad 3: A14 -> ~{A14}
- U8 pad 4: Net-(U8-Pad4) -> ~{A15}
- U8 pad 5: Net-(U16-OE#) -> CLK
- U8 pad 6: Net-(U16-OE#) -> Net-(U16-CE#)
- U8 pad 7: GND -> VCC
- U8 pad 8: R/~{W} -> Net-(U10-Cp)
- U8 pad 9: Net-(U6-P=R) -> CLK
- U9 pad 1: Net-(U8-Pad10) -> Net-(U7-Pad8)
- U9 pad 10: CLK -> GND
- U9 pad 11: Net-(U16-OE#) -> unconnected-(U9-Pad11)
- U9 pad 12: Net-(U8-Pad1) -> GND
- U9 pad 13: A15 -> GND
- U9 pad 2: CLK -> R/~{W}
- U9 pad 3: Net-(U11-Cp) -> Net-(U13-CE)
- U9 pad 4: Net-(U8-Pad13) -> Net-(U7-Pad6)
- U9 pad 6: Net-(U13-CE) -> Net-(U12-CE)
- U9 pad 8: Net-(U16-CE#) -> unconnected-(U9-Pad8)
- U9 pad 9: Net-(U8-Pad4) -> GND
Routing:
- net CLK: track 509.8 -> 507.3 mm

Commit message: Revising SDCARD board
Routing:
- net GND: track 1823.6 -> 1833.5 mm
Changed lines of the file:
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@@
-	)
-	(segment
-		(start 181.975 141.24)
-		(end 182.88 140.335)
-		(width 1)
-		(layer "F.Cu")
-		(net 1)
 	)
 	(segment
@@
 	)
 	(segment
-		(start 147.32 140.335)
-		(end 147.32 132.04)
-		(width 1)
-		(layer "F.Cu")
-		(net 1)
-	)
-	(segment
 		(start 48.895 125.095)
 		(end 50.165 126.365)
@@
 	)
 	(segment
+		(start 181.015 132.04)
+		(end 182.88 132.04)
+		(width 1)
+		(layer "F.Cu")
+		(net 1)
+	)
+	(segment
 		(start 203.195 130.17)
 		(end 202.565 129.54)
@@
 	)
 	(segment
-		(start 111.49 141.24)
-		(end 146.415 141.24)
-		(width 1)
-		(layer "F.Cu")
-		(net 1)
-	)
-	(segment
 		(start 247.96 83.415)
 		(end 246.46 81.915)
@@
 	(segment
 		(start 146.415 141.24)
-		(end 147.32 140.335)
+		(end 179.07 141.24)
 		(width 1)
 		(layer "F.Cu")
@@
 	)
 	(segment
-		(start 182.88 140.335)
-		(end 182.88 132.04)
-		(width 1)
-		(layer "F.Cu")
-		(net 1)
-	)
-	(segment
 		(start 266.065 33.655)
 		(end 264.16 31.75)
@@
 	)
 	(segment
-		(start 146.415 141.24)
-		(end 181.975 141.24)
-		(width 1)
-		(layer "F.Cu")
-		(net 1)
-	)
-	(segment
 		(start 147.32 117.475)
 		(end 147.32 119.34)
@@
 	)
 	(segment
+		(start 144.185 132.04)
+		(end 143.51 132.715)
+		(width 0.5)
+		(layer "F.Cu")
+		(net 1)
+	)
+	(segment
 		(start 123.785 87.59)
 		(end 86.36 87.59)
@@
 	)
 	(segment
+		(start 143.51 141.24)
+		(end 146.415 141.24)
+		(width 1)
+		(layer "F.Cu")
+		(net 1)
+	)
+	(segment
 		(start 147.32 105.41)
 		(end 147.32 106.64)
@@
 	)
 	(segment
+		(start 179.07 133.985)
+		(end 181.015 132.04)
+		(width 1)
+		(layer "F.Cu")
+		(net 1)
+	)
+	(segment
 		(start 57.785 67.31)
 		(end 57.15 67.945)
@@
 	)
 	(segment
+		(start 179.07 141.24)
+		(end 181.975 141.24)
+		(width 1)
+		(layer "F.Cu")
+		(net 1)
+	)
+	(segment
 		(start 162.56 29.21)
 		(end 161.925 29.845)
@@
 	)
 	(segment
+		(start 147.32 132.04)
+		(end 144.185 132.04)
+		(width 0.5)
+		(layer "F.Cu")
+		(net 1)
+	)
+	(segment
 		(start 175.26 95.24)
 		(end 175.26 92.71)
@@
 	)
 	(segment
+		(start 179.07 141.24)
+		(end 179.07 133.985)
+		(width 1)
+		(layer "F.Cu")
+		(net 1)
+	)
+	(segment
 		(start 240.03 29.21)
 		(end 238.76 30.48)
@@
 	)
 	(segment
+		(start 111.49 141.24)
+		(end 143.51 141.24)
+		(width 1)
+		(layer "F.Cu")
+		(net 1)
+	)
+	(segment
 		(start 48.895 101.6)
 		(end 48.895 112.395)
@@
 	)
 	(segment
+		(start 143.51 132.715)
+		(end 143.51 141.24)
+		(width 0.5)
+		(layer "F.Cu")
+		(net 1)
+	)
+	(segment
 		(start 202.565 116.84)
 		(end 183.515 116.84)
@@
 	)
 	(segment
+		(start 144.145 132.08)
+		(end 139.7 132.08)
+		(width 0.5)
+		(layer "F.Cu")
+		(net 1)
+	)
+	(segment
 		(start 270.875 129.54)
 		(end 271.51 130.175)
@@
 		(width 0.5)
 		(layer "F.Cu")
+		(net 1)
+	)
+	(segment
+		(start 144.185 132.04)
+		(end 144.145 132.08)
+		(width 0.5)
+		(layer "F.Cu")

Commit message: Interim commit
Routing:
- net D5: track 0.00 -> 539.1 mm, vias 0 -> 5
- net ~{RES}: track 0.00 -> 526.5 mm, vias 0 -> 3
- net D6: track 0.00 -> 524.0 mm, vias 0 -> 6
- net D3: track 0.00 -> 523.2 mm, vias 0 -> 4
- net D4: track 0.00 -> 521.2 mm, vias 0 -> 5
- net D2: track 0.00 -> 498.6 mm, vias 0 -> 3
- net D7: track 0.00 -> 494.3 mm, vias 0 -> 7
- net D0: track 0.00 -> 482.4 mm, vias 0 -> 4
- net D1: track 0.00 -> 481.7 mm, vias 0 -> 5
- net A0: track 0.00 -> 438.2 mm, vias 0 -> 6
- net R/~{W}: track 0.00 -> 419.8 mm, vias 0 -> 1
- net A2: track 0.00 -> 413.8 mm, vias 0 -> 6
- net ~{NMI}: track 0.00 -> 408.0 mm, vias 0 -> 3
- net A3: track 0.00 -> 407.6 mm, vias 0 -> 6
- net A4: track 0.00 -> 400.6 mm, vias 0 -> 3
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