File: pcb/propeller-vga/propeller-vga.kicad_sch (KiCad schematic)
At the start: 36 parts, among them J1 USB_A, J2 PPRG, J3 SER, J4 VGA, SW1 SW_Push, U1 P8X32A-D40, U2 24LC256, U3 LD1117S33TR_SOT223, Y1 5MHz

Commit message: Updating schematic
Other:
- note added: "Schematic was based on design from: https://github.com/maccasoft/propeller-vt100-terminal"
- title: (none) -> Propeller VGA board for ByteCradle 6502 / Prototype
Changed lines of the file:
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@@
 	(generator_version "8.0")
 	(paper "A4")
+	(title_block
+		(title "Propeller VGA board for ByteCradle 6502 / Prototype")
+		(date "2025-02-08")
+		(rev "0")
+	)
 	(junction
 		(at 158.75 80.01)
@@
 		)
 	)
+	(text "Schematic was based on design from:\nhttps://github.com/maccasoft/propeller-vt100-terminal"
+		(exclude_from_sim no)
+		(at 178.054 163.322 0)
+		(effects
+			(font
+				(size 1.27 1.27)
+			)
+			(justify left)
+		)
+	)
