File: pcb/propeller-vga-board/propeller-vga-board.kicad_pcb (KiCad board)
At the start: 2 copper layers, 39 parts, among them J2 PPRG, J4 VGA, J5 EXPBUS2, SW1 SW_Push, U1 P8X32A-D40, U2 24LC256, U3 LD1117S33TR_SOT223, U8 74HC138, Y1 5MHz

Commit message: Refining VGA board
Parts:
- removed J4: VGA, components:618015330923
- removed J5: EXPBUS2, Connector_PinSocket_2.54mm:PinSocket_2x20_P2.54mm_Horizontal
- removed R20: 10k, Resistor_THT:R_Axial_DIN0207_L6.3mm_D2.5mm_P7.62mm_Horizontal
- added J1: EXPBUS2, Connector_PinSocket_2.54mm:PinSocket_2x20_P2.54mm_Horizontal, F.Cu at (101.6, 144.8)
- added J3: PPRG, Connector_PinSocket_2.54mm:PinSocket_1x05_P2.54mm_Vertical, F.Cu at (125.7, 67.3)
- added R3: 4.7k, Resistor_THT:R_Axial_DIN0207_L6.3mm_D2.5mm_P7.62mm_Horizontal, F.Cu at (128.3, 86.4)
- added U4: 74HC138, Package_DIP:DIP-16_W7.62mm_Socket, F.Cu at (149.9, 81.2)
- added U5: LD1117S33TR_SOT223, Package_TO_SOT_SMD:SOT-223-3_TabPin2, F.Cu at (136.6, 88.9)
- added U6: 74HC27, Package_DIP:DIP-14_W7.62mm_Socket, F.Cu at (121.9, 81.3)
- added U7: 74HCT245, Package_DIP:DIP-20_W7.62mm_Socket, F.Cu at (128.3, 139.7)
- added U9: 74HC273, Package_DIP:DIP-20_W7.62mm_Socket, F.Cu at (92.7, 139.7)
- C3: value 10uF -> C; footprint Capacitor_THT:CP_Radial_D5.0mm_P2.50mm -> Capacitor_THT:C_Disc_D5.0mm_W2.5mm_P5.00mm
- C6: value C -> 10uF; footprint Capacitor_THT:C_Disc_D5.0mm_W2.5mm_P5.00mm -> Capacitor_THT:CP_Radial_D5.0mm_P2.50mm
- J2: value PPRG -> VGA; footprint Connector_PinSocket_2.54mm:PinSocket_1x05_P2.54mm_Vertical -> components:618015330923
- R1, R2: value 47 -> 3.9k
- R13: value 510 -> 130
- R14: value 240 -> 130
- R16, R17: value 130 -> 10k
- R4: value 10k -> 4.7k
- R5, R6: value 4.7k -> 240
- R7: value 240 -> 510
- RN1, RN2: value 1k -> 3.9k
- U1: value P8X32A-D40 -> 24LC256; footprint Package_DIP:DIP-40_W15.24mm_Socket -> Package_DIP:DIP-8_W7.62mm_Socket
- U2: value 24LC256 -> P8X32A-D40; footprint Package_DIP:DIP-8_W7.62mm_Socket -> Package_DIP:DIP-40_W15.24mm_Socket
- U3: value LD1117S33TR_SOT223 -> 74AC688; footprint Package_TO_SOT_SMD:SOT-223-3_TabPin2 -> Package_DIP:DIP-20_W7.62mm_Socket
- U8: value 74HC138 -> 74HC74; footprint Package_DIP:DIP-16_W7.62mm_Socket -> Package_DIP:DIP-14_W7.62mm_Socket
- moved C10 107.6 mm to (123.2, 133.3), turned to -90 degrees
- moved C6 104.0 mm to (149.9, 88.9), turned to 90 degrees
- moved C9 98.5 mm to (87.6, 133.4), turned to -90 degrees
- moved C5 94.1 mm to (144.8, 75.0), turned to -90 degrees
- moved RN2 93.0 mm to (122.0, 125.7)
- moved U8 90.2 mm to (86.4, 110.5)
- moved LS1 89.2 mm to (102.9, 77.5)
- moved RN1 86.1 mm to (99.1, 125.7)
- moved R9 86.1 mm to (160.0, 137.2), turned to 0 degrees
- moved U2 84.3 mm to (101.6, 118.1), turned to 90 degrees
- moved J2 82.5 mm to (189.2, 109.4)
- moved R10 81.2 mm to (160.0, 133.3), turned to 0 degrees
- moved C7 80.5 mm to (92.6, 105.4), turned to 180 degrees
- moved R11 76.3 mm to (160.0, 129.5), turned to 0 degrees
- moved C2 71.6 mm to (100.3, 90.2), turned to -90 degrees
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Connections:
- net Net-(J1-D-) renamed BIT
- C4 pad 1: +3V3 -> +5V
- C6 pad 1: +5V -> +3V3
- J2 pad 1: +3V3 -> R
- J2 pad 2: ~{RES} -> G
- J2 pad 3: RX -> B
- J2 pad 4: TX -> unconnected-(J2-Pad4)
- LS1 pad 1: Net-(U1-P14) -> Net-(U2-P14)
- LS1 pad 2: Net-(U1-P15) -> Net-(U2-P15)
- R1 pad 1: Net-(J1-D+) -> REC
- R1 pad 2: Net-(U1-P0) -> Net-(U2-P8)
- R10 pad 1: Net-(U1-P19) -> Net-(U2-P21)
- R10 pad 2: B -> G
- R11 pad 1: Net-(U1-P20) -> Net-(U2-P22)
- R11 pad 2: G -> R
- R12 pad 1: Net-(U1-P21) -> Net-(U2-P23)
- R12 pad 2: G -> R
- R13 pad 1: Net-(U1-P22) -> B
- R13 pad 2: R -> GND
- R14 pad 1: Net-(U1-P23) -> G
- R14 pad 2: R -> GND
- R15 pad 1: B -> R
- R16 pad 1: G -> +3V3
- R16 pad 2: GND -> RX
- R17 pad 1: R -> +3V3
- R17 pad 2: GND -> ~{RES}
- R2 pad 2: Net-(U1-P1) -> Net-(U2-P10)
- R4 pad 2: RX -> SCL
- R5 pad 1: +3V3 -> Net-(U2-P16)
- R5 pad 2: SDA -> VSYNC
- R6 pad 1: +3V3 -> Net-(U2-P17)
- R6 pad 2: SCL -> HSYNC
- R7 pad 1: Net-(U1-P16) -> Net-(U2-P18)
- R7 pad 2: VSYNC -> B
- R8 pad 1: Net-(U1-P17) -> Net-(U2-P19)
- R8 pad 2: HSYNC -> B
- R9 pad 1: Net-(U1-P18) -> Net-(U2-P20)
- R9 pad 2: B -> G
- RN1 pad 1: BF4 -> BF0
- RN1 pad 3: BF5 -> BF1
- RN1 pad 5: BF6 -> BF2
- RN1 pad 7: BF7 -> BF3
- RN2 pad 1: BF0 -> BF4
- RN2 pad 3: BF1 -> BF5
- RN2 pad 5: BF2 -> BF6
- RN2 pad 7: BF3 -> BF7
- U1 pad 1: Net-(RN2A-R1.2) -> GND
- U1 pad 2: Net-(RN2B-R2.2) -> GND
- U1 pad 3: Net-(RN2C-R3.2) -> GND
- U1 pad 4: Net-(RN2D-R4.2) -> GND
- U1 pad 5: Net-(RN1A-R1.2) -> SDA
- U1 pad 6: Net-(RN1B-R2.2) -> SCL
- U1 pad 7: Net-(RN1C-R3.2) -> GND
- U1 pad 8: Net-(RN1D-R4.2) -> +3V3
- U2 pad 1: GND -> Net-(RN1A-R1.2)
- U2 pad 2: GND -> Net-(RN1B-R2.2)
- U2 pad 3: GND -> Net-(RN1C-R3.2)
- U2 pad 4: GND -> Net-(RN1D-R4.2)
- U2 pad 5: SDA -> Net-(RN2A-R1.2)
- U2 pad 6: SCL -> Net-(RN2B-R2.2)
- U2 pad 7: GND -> Net-(RN2C-R3.2)
- U2 pad 8: +3V3 -> Net-(RN2D-R4.2)
- U3 pad 1: GND -> ~{I/O}
- U3 pad 2: +3V3 -> GND
- U3 pad 3: +5V -> GND
- U8 pad 1: A0 -> +5V
- U8 pad 10: unconnected-(U8-~{Y5}-Pad10) -> +5V
- U8 pad 11: unconnected-(U8-~{Y4}-Pad11) -> Net-(U8B-C)
- U8 pad 12: ~{SETBIT} -> D0
- U8 pad 13: ~{STATUS} -> ~{RES}
- U8 pad 14: ~{SETREC} -> +5V
- U8 pad 2: A1 -> unconnected-(U8A-D-Pad2)
- U8 pad 4: Net-(U4-P=R) -> +5V
- U8 pad 5: Net-(U4-P=R) -> unconnected-(U8A-Q-Pad5)
- U8 pad 6: +5V -> unconnected-(U8A-~{Q}-Pad6)
- U8 pad 7: unconnected-(U8-~{Y7}-Pad7) -> GND
- U8 pad 8: GND -> unconnected-(U8B-~{Q}-Pad8)
- U8 pad 9: unconnected-(U8-~{Y6}-Pad9) -> REC
- Y1 pad 1: Net-(U1-XI) -> Net-(U2-XI)
- Y1 pad 2: Net-(U1-XO) -> Net-(U2-XO)
Routing:
- net +5V: track 107.7 -> 522.0 mm, vias 0 -> 1
- net GND: track 372.1 -> 730.0 mm, vias 1 -> 0
- net A0: track 0.00 -> 135.7 mm, vias 0 -> 1
- net A1: track 0.00 -> 117.9 mm, vias 0 -> 2
- net R/~{W}: track 0.00 -> 116.0 mm, vias 0 -> 3
- net ~{I/O}: track 0.00 -> 105.9 mm, vias 0 -> 2
- net CLK: track 0.00 -> 104.4 mm
- net Net-(U3-P=R): track 0.00 -> 80.0 mm, vias 0 -> 1
- net D0: track 0.00 -> 79.3 mm
- net A3: track 0.00 -> 77.6 mm
- net Net-(U2-P14): track 0.00 -> 75.8 mm, vias 0 -> 1
- net Net-(U8B-C): track 0.00 -> 74.4 mm
- net D7: track 0.00 -> 74.3 mm
- net A7: track 0.00 -> 73.8 mm
- net ~{STATUS}: track 0.00 -> 72.1 mm
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- added copper zone on B.Cu, net +5V
- added copper zone on F.Cu, net GND
Other:
- board outline added: 106.7 x 85.8 mm
- board text added: "Parallax Propeller VGA Interface Board"
- board text removed: "5V"

Commit message: Removing bitpin
Parts:
- removed R2: 3.9k, Resistor_THT:R_Axial_DIN0207_L6.3mm_D2.5mm_P7.62mm_Horizontal
Connections:
- U2 pad 15: Net-(U2-P10) -> unconnected-(U2-P10-Pad15)
- U4 pad 12: ~{SETBIT} -> unconnected-(U4-~{Y3}-Pad12)
Routing:
- net Net-(U2-P10): track 18.7 -> 0.00 mm
