File: pcb/propeller-vga-board/propeller-vga-board.kicad_sch (KiCad schematic)
At the start: 44 parts, among them J2 PPRG, J4 VGA, J5 EXPBUS2, SW1 SW_Push, U1 P8X32A-D40, U2 24LC256, U3 LD1117S33TR_SOT223, U4 74HC688, U5 74HC273, U6 74HC74, U7 74LS10, U8 74HC138, U9 74HCT245, Y1 5MHz

Commit message: Refining VGA board
Parts:
- removed U7: 74LS10, Package_DIP:DIP-14_W7.62mm_Socket, symbol 74xx:74LS10
- added U6: 74HC27, Package_DIP:DIP-14_W7.62mm_Socket, symbol 74xx:74LS27
- R1, R2: value 1k -> 3.9k
- RN1: renamed from RN2; value 1k -> 3.9k
- RN2: renamed from RN1; value 1k -> 3.9k
- U3: renamed from U4; value 74HC688 -> 74AC688
- renumbered C4 to C1, C8 to C10, C1 to C2, C2 to C3, C5 to C4, C6 to C5, C3 to C6, C9 to C7, C7 to C8, C10 to C9, J5 to J1, J4 to J2, J2 to J3, R12 to R10, R13 to R11, R14 to R12, R15 to R13, R16 to R14, R17 to R15, R4 to R16, R20 to R17, R5 to R3, R6 to R4, R7 to R5, R8 to R6, R9 to R7, R10 to R8, R11 to R9, U2 to U1, U1 to U2, U8 to U4, U3 to U5, U9 to U7, U6 to U8, U5 to U9
Connections:
- net +5V: now also U8.1 (~{R}), U6.14 (VCC)
- net BIT: no longer U8.5 (Q)
- net CLK: now also U6.10, U6.11, U6.9
- net D0: no longer U8.2 (D)
- net GND: now also U8.3 (C), U6.7 (GND)
- net R/~{W}: now also U6.2, U6.4
- net ~{DATA}: now also U6.1
- net ~{RES}: no longer U8.1 (~{R})
- net ~{SETREC}: now also U6.3
- net at U9.11 (Cp): now also U6.12
- net at U8.11 (C): now also U6.6
- new net ~{CLK}: U6.13, U6.5, U6.8
- no-connect marks 19 -> 21
Other:
- moved on the sheet: C1, C10, C2, C3, C4, C5, C6, C7, C8, C9, J1, J2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

Commit message: Removing bitpin
Parts:
- removed R2: 3.9k, Resistor_THT:R_Axial_DIN0207_L6.3mm_D2.5mm_P7.62mm_Horizontal, symbol Device:R
Connections:
- net ~{SETBIT}: no longer names the net of U4.12 (~{Y3})
- no-connect marks 21 -> 23
Changed lines of the file:
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@@
 	)
 	(no_connect
+		(at 119.38 144.78)
+	)
+	(no_connect
 		(at 116.84 114.3)
 	)
@@
 	)
 	(no_connect
+		(at 50.8 71.12)
+	)
+	(no_connect
 		(at 119.38 152.4)
 	)
@@
 	(wire
 		(pts
-			(xy 33.02 71.12) (xy 50.8 71.12)
-		)
-		(stroke
-			(width 0)
-			(type default)
-		)
-	)
-	(wire
-		(pts
 			(xy 39.37 60.96) (xy 50.8 60.96)
 		)
@@
 	(wire
 		(pts
-			(xy 29.21 81.28) (xy 33.02 81.28)
-		)
-		(stroke
-			(width 0)
-			(type default)
-		)
-	)
-	(wire
-		(pts
 			(xy 38.1 50.8) (xy 38.1 53.34)
 		)
@@
 	(wire
 		(pts
-			(xy 33.02 81.28) (xy 33.02 71.12)
-		)
-		(stroke
-			(width 0)
-			(type default)
-		)
-	)
-	(wire
-		(pts
 			(xy 86.36 137.16) (xy 90.17 137.16)
 		)
@@
 		)
 	)
-	(global_label "~{SETBIT}"
-		(shape input)
-		(at 119.38 144.78 0)
-		(fields_autoplaced yes)
-		(effects
-			(font
-				(size 1.27 1.27)
-			)
-			(justify left)
-		)
-		(property "Intersheetrefs" "${INTERSHEET_REFS}"
-			(at 128.5337 144.78 0)
-			(effects
-				(font
-					(size 1.27 1.27)
-				)
-				(justify left)
-				(hide yes)
-			)
-		)
-	)
 	(global_label "~{I{slash}O}"
 		(shape input)
@@
 		)
 	)
-	(global_label "BIT"
-		(shape input)
-		(at 21.59 81.28 180)
-		(fields_autoplaced yes)
-		(effects
-			(font
-				(size 1.27 1.27)
-			)
-			(justify right)
-		)
-		(property "Intersheetrefs" "${INTERSHEET_REFS}"
-			(at 15.7624 81.28 0)
-			(effects
-				(font
-					(size 1.27 1.27)
-				)
-				(justify right)
-				(hide yes)
-			)
-		)
-	)
 	(global_label "BF3"
 		(shape input)
@@
 					(unit 1)
 				)
-			)
-		)
-	)
-	(symbol
-		(lib_id "Device:R")
-		(at 25.4 81.28 90)
-		(unit 1)
-		(exclude_from_sim no)
-		(in_bom yes)
-		(on_board yes)
-		(dnp no)
-		(property "Reference" "R2"
-			(at 25.4 78.994 90)
-			(effects
-				(font
-					(size 1.27 1.27)
-				)
-			)
-		)
-		(property "Value" "3.9k"
-			(at 25.4 81.28 90)
-			(effects
-				(font
-					(size 1.27 1.27)
-				)
-			)
-		)
-		(property "Footprint" "Resistor_THT:R_Axial_DIN0207_L6.3mm_D2.5mm_P7.62mm_Horizontal"
-			(at 25.4 83.058 90)
-			(effects
-				(font
-					(size 1.27 1.27)
-				)
-				(hide yes)
-			)
-		)
-		(property "Datasheet" "~"
-			(at 25.4 81.28 0)
-			(effects
-				(font
-					(size 1.27 1.27)
-				)
-				(hide yes)
-			)
-		)
-		(property "Description" "Resistor"
-			(at 25.4 81.28 0)
-			(effects
-				(font
-					(size 1.27 1.27)
-				)
-				(hide yes)
-			)
-		)
-		(pin "2"
-		)
-		(pin "1"
-		)
-		(instances
-			(project "propeller-vga-board"
-				(path "/68d9e336-094e-4def-a139-3412ac01f132"
-					(reference "R2")
-					(unit 1)
-				)
