File: pcb/sdcard-board/sdcard-board.kicad_sch (KiCad schematic)
At the start: 39 parts, among them J3 SD Card Board, J4 EXPBUS1, U1 74HC123, U10 74HC138, U3 74HC00, U4 74HC00, U5 74HC163, U6 74HC00, U7 74HC165, U8 74HC595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

Commit message: Further redesigning boards
Parts:
- removed C3: 220uF, Capacitor_THT:CP_Radial_D6.3mm_P2.50mm, symbol Device:C_Polarized
- removed J4: EXPBUS1, Connector_PinHeader_2.54mm:PinHeader_2x20_P2.54mm_Vertical, symbol Connector_Generic:Conn_02x20_Counter_Clockwise
- added C13, C3: 0.1uF, Capacitor_THT:C_Disc_D5.0mm_W2.5mm_P5.00mm, symbol Device:C
- added J1: EXPBUS2, Connector_PinSocket_2.54mm:PinSocket_2x20_P2.54mm_Horizontal, symbol Connector_Generic:Conn_02x20_Odd_Even
- J3: footprint Connector_PinSocket_2.54mm:PinSocket_1x06_P2.54mm_Vertical -> sdcard-holder:sdcard-socket
- TP5, TP6, TP7, TP8: footprint TestPoint:TestPoint_Pad_4.0x4.0mm -> TestPoint:TestPoint_THTPad_2.5x2.5mm_Drill1.2mm
- U10: footprint (none) -> Package_DIP:DIP-16_W7.62mm_Socket
- U9: footprint (none) -> Package_DIP:DIP-20_W7.62mm_Socket
Connections:
- net A0: now also J1.3 (Pin_3)
- net A1: now also J1.5 (Pin_5)
- net A10: now also J1.23 (Pin_23)
- net A11: now also J1.25 (Pin_25)
- net A12: now also J1.27 (Pin_27)
- net A13: now also J1.29 (Pin_29)
- net A14: now also J1.31 (Pin_31)
- net A15: now also J1.33 (Pin_33)
- net A2: now also J1.7 (Pin_7)
- net A3: now also J1.9 (Pin_9)
- net A4: now also J1.11 (Pin_11)
- net A5: now also J1.13 (Pin_13)
- net A6: now also J1.15 (Pin_15)
- net A7: now also J1.17 (Pin_17)
- net A8: now also J1.19 (Pin_19)
- net A9: now also J1.21 (Pin_21)
- net CLK: now also J1.6 (Pin_6)
- net D0: now also J1.24 (Pin_24)
- net D1: now also J1.26 (Pin_26)
- net D2: now also J1.28 (Pin_28)
- net D3: now also J1.30 (Pin_30)
- net D4: now also J1.32 (Pin_32)
- net D5: now also J1.34 (Pin_34)
- net D6: now also J1.36 (Pin_36)
- net D7: now also J1.38 (Pin_38)
- net GND: now also C13.2, C3.2, J1.39 (Pin_39), J1.40 (Pin_40)
- net R/~{W}: now also J1.4 (Pin_4)
- net VCC: now also C13.1, C3.1, J1.1 (Pin_1), J1.2 (Pin_2)
- net ~{IRQ}: now also J1.14 (Pin_14)
- net ~{I/O}: now also J1.18 (Pin_18)
- net ~{NMI}: now also J1.12 (Pin_12)
- net ~{RES}: now also J1.10 (Pin_10)
Other:
- note added: "0x7F20-0x7F23"
- moved on the sheet: C10, C11, C12, C4, C5, C6, C7, C8, C9, U1C, U3E, U4E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

Commit message: Revising SDCARD board
Connections:
- net CLK: now also U6.12; no longer J3.2 (Pin_2), TP3.1, U3.12, U3.13, U5.14 (Q0), U8.11 (SRCLK)
- net SD_SPI: now also U6.4
- net VCC: no longer U6.12, U6.13
- net ~{SER_WR}: now also U6.10, U6.9; no longer U7.1 (~{PL})
- net at U6.8: now also U6.13; no longer D2.1 (K)
- net at U6.11: now also U7.1 (~{PL})
- net ~{CLK} renamed ~{SDCLK}
- new net: D2.1 (K), U6.3
- new net SDCLK: J3.2 (Pin_2), TP3.1, U3.12, U3.13, U5.14 (Q0), U8.11 (SRCLK)
Other:
- moved on the sheet: D2, R3, TP1, TP2, TP3, TP4, TP5, TP6, TP7, TP8, U3D, U6C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

Commit message: Initial commit bitbang SD-card routines
Changed lines of the file:
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@@
 (kicad_sch
-	(version 20231120)
+	(version 20250114)
 	(generator "eeschema")
-	(generator_version "8.0")
+	(generator_version "9.0")
 	(paper "A3")
 	(title_block
 		(date "2025-01-24")
 	)
+	(text "SHIFT REGISTER SD -> Z80\nIN REGISTER"
+		(exclude_from_sim no)
+		(at 176.53 82.55 0)
+		(effects
+			(font
+				(size 1.27 1.27)
+			)
+			(justify left bottom)
+		)
+	)
+	(text "SD CARD\nS/R LATCHES"
+		(exclude_from_sim no)
+		(at 16.51 139.065 0)
+		(effects
+			(font
+				(size 1.27 1.27)
+			)
+			(justify left bottom)
+		)
+	)
+	(text "out $00: ~{SER_WR} is pulled low, loading the values on the data bus into the out register.\nout $01: ~{CLKSTART} is pulled low, starting the counter circuit and pushing a byte into \n         the SD card while simultaneously reading a byte.\nout $02: ~{SDCS_SET} is pulled low, pulling ~{CS} low, activating the SD card.\nout $03: ~{SDCS_RESET} is pulled low, pulling ~{CS} high, deactivating the SD card."
+		(exclude_from_sim no)
+		(at 287.528 107.061 0)
+		(effects
+			(font
+				(size 1.27 1.27)
+			)
+			(justify left bottom)
+		)
+	)
+	(text "On ~{CLKSTART}, this component produces exactly\n8 pulses at 8MHz."
+		(exclude_from_sim no)
+		(at 27.305 29.21 0)
+		(effects
+			(font
+				(size 1.27 1.27)
+			)
+			(justify left bottom)
+		)
+	)
+	(text "On ~{CLKSTART}, \n~{MR} will be set HIGH, \nactivating the counter."
+		(exclude_from_sim no)
+		(at 20.32 67.31 0)
+		(effects
+			(font
+				(size 1.27 1.27)
+			)
+			(justify left bottom)
+		)
+	)
+	(text "in $00: ~{SER_RD} is pulled low, reading from the in register.\nin $01: Does nothing\nin $02: ~{SDOUT_SET} is pulled low, pulling MISO low via a 10k resistor.\nin $03: ~{SDOUT_RESET} is pulled low, pulling MISO high via a 10k resistor.\n\nWhen no card is present, the output of the SD card will follow the output of the SET/RESET latch,\nhowever if a card is present, though unresponsive, it will not follow and the same (high) output\nwill be received."
+		(exclude_from_sim no)
+		(at 287.528 125.476 0)
+		(effects
+			(font
+				(size 1.27 1.27)
+			)
+			(justify left bottom)
+		)
+	)
+	(text "0x7F20-0x7F23"
+		(exclude_from_sim no)
+		(at 322.326 28.956 0)
+		(effects
+			(font
+				(size 1.27 1.27)
+			)
+		)
+	)
+	(text "SELECTION COMPONENT"
+		(exclude_from_sim no)
+		(at 254 18.796 0)
+		(effects
+			(font
+				(size 1.27 1.27)
+			)
+			(justify left bottom)
+		)
+	)
+	(text "1k resistor with 22pF cap gives\n0.45*RC = 0.01us active low pulse"
+		(exclude_from_sim no)
+		(at 241.3 130.81 0)
+		(effects
+			(font
+				(size 1.27 1.27)
+			)
+			(justify left bottom)
+		)
+	)
+	(text "10k resistor with 22pF cap gives\nt = 0.45RC = 0.1us delay between consecutive pulses"
+		(exclude_from_sim no)
+		(at 170.815 125.095 0)
+		(effects
+			(font
+				(size 1.27 1.27)
+			)
+			(justify left bottom)
+		)
+	)
+	(text "CLOCK COMPONENT"
+		(exclude_from_sim no)
+		(at 16.51 18.415 0)
+		(effects
+			(font
+				(size 1.27 1.27)
+			)
+			(justify left bottom)
+		)
+	)
+	(text "INTERFACE PORTS"
+		(exclude_from_sim no)
+		(at 120.015 80.01 0)
+		(effects
+			(font
+				(size 1.27 1.27)
+			)
+			(justify left bottom)
+		)
+	)
+	(text "Both CEP and CET need\nto be high for count\nto be enabled."
+		(exclude_from_sim no)
+		(at 50.8 68.58 0)
+		(effects
+			(font
+				(size 1.27 1.27)
+			)
+			(justify left bottom)
+		)
+	)
+	(text "SCK"
+		(exclude_from_sim no)
+		(at 256.54 100.076 0)
+		(effects
+			(font
+				(size 1 1)
+			)
+			(justify left bottom)
+		)
+	)
+	(text "MULTIVIBRATOR DELAY COMPONENT"
+		(exclude_from_sim no)
+		(at 173.99 120.65 0)
+		(effects
+			(font
+				(size 1.27 1.27)
+			)
+			(justify left bottom)
+		)
+	)
+	(text "SHIFT REGISTER Z80 -> SD\nOUT REGISTER"
+		(exclude_from_sim no)
+		(at 177.165 20.955 0)
+		(effects
+			(font
+				(size 1.27 1.27)
+			)
+			(justify left bottom)
+		)
+	)
 	(junction
 		(at 360.68 48.26)
@@
 		)
 	)
-	(text "SHIFT REGISTER SD -> Z80\nIN REGISTER"
-		(exclude_from_sim no)
-		(at 176.53 82.55 0)
-		(effects
-			(font
-				(size 1.27 1.27)
-			)
-			(justify left bottom)
-		)
-	)
-	(text "SD CARD\nS/R LATCHES"
-		(exclude_from_sim no)
-		(at 16.51 139.065 0)
-		(effects
-			(font
-				(size 1.27 1.27)
-			)
-			(justify left bottom)
-		)
-	)
-	(text "out $00: ~{SER_WR} is pulled low, loading the values on the data bus into the out register.\nout $01: ~{CLKSTART} is pulled low, starting the counter circuit and pushing a byte into \n         the SD card while simultaneously reading a byte.\nout $02: ~{SDCS_SET} is pulled low, pulling ~{CS} low, activating the SD card.\nout $03: ~{SDCS_RESET} is pulled low, pulling ~{CS} high, deactivating the SD card."
-		(exclude_from_sim no)
-		(at 287.528 107.061 0)
-		(effects
-			(font
-				(size 1.27 1.27)
-			)
-			(justify left bottom)
-		)
-	)
-	(text "On ~{CLKSTART}, this component produces exactly\n8 pulses at 8MHz."
-		(exclude_from_sim no)
-		(at 27.305 29.21 0)
-		(effects
-			(font
-				(size 1.27 1.27)
-			)
-			(justify left bottom)
-		)
-	)
-	(text "On ~{CLKSTART}, \n~{MR} will be set HIGH, \nactivating the counter."
-		(exclude_from_sim no)
-		(at 20.32 67.31 0)
-		(effects
-			(font
-				(size 1.27 1.27)
-			)
-			(justify left bottom)
-		)
-	)
-	(text "in $00: ~{SER_RD} is pulled low, reading from the in register.\nin $01: Does nothing\nin $02: ~{SDOUT_SET} is pulled low, pulling MISO low via a 10k resistor.\nin $03: ~{SDOUT_RESET} is pulled low, pulling MISO high via a 10k resistor.\n\nWhen no card is present, the output of the SD card will follow the output of the SET/RESET latch,\nhowever if a card is present, though unresponsive, it will not follow and the same (high) output\nwill be received."
-		(exclude_from_sim no)
-		(at 287.528 125.476 0)
-		(effects
-			(font
-				(size 1.27 1.27)
-			)
-			(justify left bottom)
-		)
-	)
-	(text "0x7F20-0x7F23"
-		(exclude_from_sim no)
-		(at 322.326 28.956 0)
-		(effects
-			(font
-				(size 1.27 1.27)
-			)
-		)
-	)
-	(text "SELECTION COMPONENT"
-		(exclude_from_sim no)
-		(at 254 18.796 0)
-		(effects
-			(font
-				(size 1.27 1.27)
-			)
-			(justify left bottom)
-		)
-	)
-	(text "1k resistor with 22pF cap gives\n0.45*RC = 0.01us active low pulse"
-		(exclude_from_sim no)
-		(at 241.3 130.81 0)
-		(effects
-			(font
-				(size 1.27 1.27)
-			)
-			(justify left bottom)
-		)
-	)
-	(text "10k resistor with 22pF cap gives\nt = 0.45RC = 0.1us delay between consecutive pulses"
-		(exclude_from_sim no)
-		(at 170.815 125.095 0)
-		(effects
-			(font
-				(size 1.27 1.27)
-			)
-			(justify left bottom)
-		)
-	)
-	(text "CLOCK COMPONENT"
-		(exclude_from_sim no)
-		(at 16.51 18.415 0)
-		(effects
-			(font
-				(size 1.27 1.27)
-			)
-			(justify left bottom)
-		)
-	)
-	(text "INTERFACE PORTS"
-		(exclude_from_sim no)
-		(at 120.015 80.01 0)
-		(effects
-			(font
-				(size 1.27 1.27)
-			)
-			(justify left bottom)
-		)
-	)
-	(text "Both CEP and CET need\nto be high for count\nto be enabled."
-		(exclude_from_sim no)
-		(at 50.8 68.58 0)
-		(effects
-			(font
-				(size 1.27 1.27)
-			)
-			(justify left bottom)
-		)
-	)
-	(text "SCK"
-		(exclude_from_sim no)
-		(at 256.54 100.076 0)
-		(effects
-			(font
-				(size 1 1)
-			)
-			(justify left bottom)
-		)
-	)
-	(text "MULTIVIBRATOR DELAY COMPONENT"
-		(exclude_from_sim no)
-		(at 173.99 120.65 0)
-		(effects
-			(font
-				(size 1.27 1.27)
-			)
-			(justify left bottom)
-		)
-	)
-	(text "SHIFT REGISTER Z80 -> SD\nOUT REGISTER"
-		(exclude_from_sim no)
-		(at 177.165 20.955 0)
-		(effects
-			(font
-				(size 1.27 1.27)
-			)
-			(justify left bottom)
-		)
-	)
 	(global_label "~{CLKSTOP}"
 		(shape input)
@@
 		)
 	)
+	(embedded_fonts no)
 )
