File: pcb/mini-board/_autosave-peripherals.kicad_sch (KiCad schematic)
At the start: 20 parts, among them J2 Conn_02x14_Odd_Even, J3 SD Card Board, J8 SERIAL, U15 SST39SF040, U16 AS6C4008-55, U19 W65C22NxP, U21 W65C51NxP, U22 MAX232, Y1 1.8432 MHz

Commit message: Initial commit miniboard revision
Parts:
- U16: footprint Package_DIP:DIP-32_W15.24mm -> Package_DIP:DIP-32_W15.24mm_Socket
- U19: footprint Package_DIP:DIP-40_W15.24mm -> Package_DIP:DIP-40_W15.24mm_Socket
- U21: footprint Package_DIP:DIP-28_W15.24mm -> Package_DIP:DIP-28_W15.24mm_Socket
Changed lines of the file:
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@@
 			)
 		)
-		(property "Footprint" "Package_DIP:DIP-28_W15.24mm"
+		(property "Footprint" "Package_DIP:DIP-28_W15.24mm_Socket"
 			(at 55.88 102.87 0)
 			(effects
@@
 			)
 		)
-		(property "Footprint" "Package_DIP:DIP-40_W15.24mm"
+		(property "Footprint" "Package_DIP:DIP-40_W15.24mm_Socket"
 			(at 179.07 13.97 0)
 			(effects
@@
 			)
 		)
-		(property "Footprint" "Package_DIP:DIP-32_W15.24mm"
+		(property "Footprint" "Package_DIP:DIP-32_W15.24mm_Socket"
 			(at 43.18 58.42 0)
 			(effects
