File: pcb/tiny-board/tiny-board.kicad_sch (KiCad schematic)
At the start: 41 parts, among them J1 USB_B, J2 SYSTEM BUS, J6 UART1, SW1 RESET, SW2 NMI, SW3 SW_SPDT, U10 ATF22V10, U11 DS1813, U2 W65C02, U5 SST39SF010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

Commit message: Making small changes to tiny board and updating documentation
Parts:
- renumbered C2 to C1, C1 to C10, C12 to C11, C18 to C12, C19 to C13, C16 to C14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
