File: pcb/daughterboards/tinyboard-blinkenlight/tinyboard-blinkenlight.kicad_pcb (KiCad board)
At the start: 2 copper layers, 38.1 x 63.5 mm, 15 parts, among them J2 SYSTEM BUS, U1 74HC273, U2 74HC02

Commit message: Adding strobe
Other:
- board size 38.1 x 63.5 mm -> 43.2 x 63.5 mm
- board text added: "VCC A0 A1 A2 A3 A4 A5 A6 A7 A8 A9 A10 A11 A12 A13 A14 A15 TxD RxD GND"
- board text added: "VCC R/~{W} CLK ~{B2} ~{B1} ~{RES} ~{NMI} ~{IRQ} ~{ROM} ~{ACIA} ~{RAM} D0 D1 D2 D3 D4 D5 D6 D7 GND"
Changed lines of the file:
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@@
 			(psa4output no)
 			(plot_black_and_white yes)
-			(plotinvisibletext no)
 			(sketchpadsonfab no)
 			(plotpadnumbers no)
@@
 		(tags "LED")
 		(property "Reference" "D5"
-			(at 1.27 -3.96 0)
+			(at 5.334 0 90)
 			(layer "F.SilkS")
 			(effects
@@
 		(tags "LED")
 		(property "Reference" "D1"
-			(at 1.27 -3.96 0)
+			(at 5.334 0 90)
 			(layer "F.SilkS")
 			(effects
@@
 		(tags "LED")
 		(property "Reference" "D7"
-			(at 1.27 -3.96 0)
+			(at 5.334 0 90)
 			(layer "F.SilkS")
 			(effects
@@
 		(tags "LED")
 		(property "Reference" "D6"
-			(at 1.27 -3.96 0)
+			(at 5.334 0 90)
 			(layer "F.SilkS")
 			(effects
@@
 		(tags "LED")
 		(property "Reference" "D8"
-			(at 1.27 -3.96 0)
+			(at 5.334 0 270)
 			(layer "F.SilkS")
 			(effects
@@
 		(tags "LED")
 		(property "Reference" "D3"
-			(at 1.27 -3.96 0)
+			(at 5.334 0 90)
 			(layer "F.SilkS")
 			(effects
@@
 		(tags "LED")
 		(property "Reference" "D4"
-			(at 1.27 -3.96 0)
+			(at 5.334 0 90)
 			(layer "F.SilkS")
 			(effects
@@
 		(tags "LED")
 		(property "Reference" "D2"
-			(at 1.27 -3.96 0)
+			(at 5.334 0 90)
 			(layer "F.SilkS")
 			(effects
@@
 		)
 		(property "Value" "SYSTEM BUS"
-			(at -5.08 44.45 90)
+			(at -1.27 50.8 180)
 			(layer "F.SilkS")
 			(effects
@@
 	)
 	(gr_arc
-		(start 69.31 88.9)
-		(mid 67.895786 88.314214)
-		(end 67.31 86.9)
+		(start 108.491016 25.4)
+		(mid 109.90487 25.985427)
+		(end 110.491015 27.398984)
 		(stroke
 			(width 0.05)
@@
 	)
 	(gr_arc
-		(start 103.41 25.4)
-		(mid 104.824214 25.985786)
-		(end 105.41 27.4)
+		(start 69.31 88.9)
+		(mid 67.895786 88.314214)
+		(end 67.31 86.9)
 		(stroke
 			(width 0.05)
@@
 		(layer "Edge.Cuts")
 	)
-	(gr_arc
-		(start 105.41 86.9)
-		(mid 104.824214 88.314214)
-		(end 103.41 88.9)
+	(gr_line
+		(start 108.521236 88.9)
+		(end 69.31 88.9)
 		(stroke
 			(width 0.05)
@@
 	)
 	(gr_line
-		(start 103.41 88.9)
-		(end 69.31 88.9)
+		(start 110.491015 27.398984)
+		(end 110.521236 86.898984)
 		(stroke
 			(width 0.05)
@@
 		(layer "Edge.Cuts")
 	)
-	(gr_line
-		(start 105.41 27.4)
-		(end 105.41 86.9)
+	(gr_arc
+		(start 110.521236 86.898984)
+		(mid 109.935811 88.313867)
+		(end 108.521236 88.9)
 		(stroke
 			(width 0.05)
@@
 	(gr_line
 		(start 69.31 25.4)
-		(end 103.41 25.4)
+		(end 108.491016 25.4)
 		(stroke
 			(width 0.05)
@@
 	)
 	(gr_text "ByteCradle 6502\nTINY BLINKENLIGHT"
-		(at 72.39 78.74 90)
+		(at 72.644 78.74 90)
 		(layer "F.SilkS")
 		(effects
 			(font
-				(size 1 1)
+				(size 1.2 1.2)
 				(thickness 0.2)
 			)
@@
 		)
 	)
+	(gr_text "VCC\nR/~{W}\nCLK\n~{B2}\n~{B1}\n~{RES}\n~{NMI}\n~{IRQ}\n~{ROM}\n~{ACIA}\n~{RAM}\nD0\nD1\nD2\nD3\nD4\nD5\nD6\nD7\nGND"
+		(at 100.33 82.296 0)
+		(layer "F.SilkS" knockout)
+		(effects
+			(font
+				(size 1.585 1)
+				(thickness 0.25)
+				(bold yes)
+			)
+			(justify right bottom)
+		)
+	)
+	(gr_text "VCC\nA0\nA1\nA2\nA3\nA4\nA5\nA6\nA7\nA8\nA9\nA10\nA11\nA12\nA13\nA14\nA15\nTxD\nRxD\nGND"
+		(at 105.47 82.296 0)
+		(layer "F.SilkS" knockout)
+		(effects
+			(font
+				(size 1.585 1)
+				(thickness 0.25)
+				(bold yes)
+			)
+			(justify left bottom)
+		)
+	)
 	(segment
 		(start 88.9 87.63)
@@
 		(polygon
 			(pts
-				(xy 66.04 24.13) (xy 106.68 24.13) (xy 106.68 90.17) (xy 66.04 90.17)
+				(xy 66.04 24.13) (xy 112.268 24.13) (xy 112.014 90.17) (xy 66.04 90.17)
 			)
 		)
@@
 		(polygon
 			(pts
-				(xy 66.04 24.13) (xy 106.68 24.13) (xy 106.68 90.17) (xy 66.04 90.17)
+				(xy 66.04 24.13) (xy 112.268 24.13) (xy 112.014 90.17) (xy 66.04 90.17)
 			)
 		)
